File: PCB/Center_Console/Center_Armament/Armament_MCU/Backlighting.kicad_sch (KiCad schematic)
At the start: 40 parts, among them J10 AUX_PANEL_BACKLIGHT_2, J7 AUX_PANEL_BACKLIGHT_3, J8 AUX_PANEL_BACKLIGHT_4, J9 AUX_PANEL_BACKLIGHT_1, Q1 IRLML2502, Q2 IRLML2502

Commit message: Switch stepper driver DRV8835 → DRV8833PW; rework IRLML2502 symbol
DRV8835 is only available in WSON-12 (bottom-terminated, not inspectable
post-reflow). Replaced throughout with DRV8833PW (HTSSOP-16) which is
already placed in Gauges.kicad_sch as the placeholder.

Library: remove DRV8835 symbol block from OpenSkyhawk.kicad_sym; rework
IRLML2502 symbol body with proper N-channel MOSFET graphical elements
(was a plain rectangle).

Docs: update hardware-standards.md stepper driver section (DRV8833PW,
VINT/VCP/AISEN/FAULT handling); update kicad.md library table; update
Center_Armament.md MCU board component list.

Schematics: KiCad project file and sub-sheets updated from Symbol Editor
session (IRLML2502 symbol refresh across Backlighting and Gauges sheets).
Parts:
- R18, R19, R20, R21: footprint (none) -> Resistor_SMD:R_0805_2012Metric
Changed lines of the file:
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@@
 	(wire
 		(pts
-			(xy 252.73 76.2) (xy 245.11 76.2)
-		)
-		(stroke
-			(width 0)
-			(type default)
-		)
-	)
-	(wire
-		(pts
 			(xy 50.8 138.43) (xy 58.42 138.43)
 		)
@@
 	(wire
 		(pts
-			(xy 250.19 58.42) (xy 250.19 52.07)
-		)
-		(stroke
-			(width 0)
-			(type default)
-		)
-	)
-	(wire
-		(pts
 			(xy 115.57 66.04) (xy 127 66.04)
 		)
@@
 	(wire
 		(pts
-			(xy 54.61 80.01) (xy 62.23 80.01)
+			(xy 245.11 78.74) (xy 245.11 85.09)
 		)
 		(stroke
@@
 	(wire
 		(pts
-			(xy 111.76 138.43) (xy 123.19 138.43)
+			(xy 54.61 80.01) (xy 62.23 80.01)
 		)
 		(stroke
@@
 	(wire
 		(pts
-			(xy 252.73 88.9) (xy 252.73 76.2)
+			(xy 111.76 138.43) (xy 123.19 138.43)
 		)
 		(stroke
@@
 	(wire
 		(pts
-			(xy 252.73 91.44) (xy 252.73 95.25)
-		)
-		(stroke
-			(width 0)
-			(type default)
-		)
-	)
-	(wire
-		(pts
-			(xy 250.19 39.37) (xy 250.19 49.53)
-		)
-		(stroke
-			(width 0)
-			(type default)
-		)
-	)
-	(wire
-		(pts
-			(xy 252.73 95.25) (xy 245.11 95.25)
+			(xy 54.61 66.04) (xy 62.23 66.04)
 		)
 		(stroke
@@
 	(wire
 		(pts
-			(xy 54.61 66.04) (xy 62.23 66.04)
+			(xy 66.04 138.43) (xy 73.66 138.43)
 		)
 		(stroke
@@
 	(wire
 		(pts
-			(xy 66.04 138.43) (xy 73.66 138.43)
+			(xy 46.99 52.07) (xy 41.91 52.07)
 		)
 		(stroke
@@
 	(wire
 		(pts
-			(xy 46.99 52.07) (xy 41.91 52.07)
+			(xy 242.57 38.1) (xy 242.57 45.72)
 		)
 		(stroke
@@
 	)
 	(label "PANEL_BACKLIGHT_RETURN"
-		(at 250.19 39.37 180)
+		(at 242.57 38.1 180)
 		(effects
 			(font
@@
 	)
 	(label "GAUGE_BACKLIGHT_RETURN"
-		(at 245.11 76.2 180)
+		(at 245.11 78.74 180)
 		(effects
 			(font
@@
 		(in_pos_files yes)
 		(dnp no)
-		(fields_autoplaced yes)
 		(property "Reference" "Q2"
-			(at 245.11 82.55 0)
+			(at 241.3 86.36 0)
 			(show_name no)
 			(do_not_autoplace no)
@@
 		)
 		(property "Value" "IRLML2502"
-			(at 245.11 85.09 0)
+			(at 248.92 90.17 90)
 			(show_name no)
 			(do_not_autoplace no)
@@
 			)
 		)
-		(property "Datasheet" "https://www.infineon.com/dgdl/irlml2502pbf.pdf"
+		(property "Datasheet" "https://www.infineon.com/assets/row/public/documents/24/49/infineon-irlml2502-datasheet-en.pdf"
 			(at 245.11 90.17 0)
 			(hide yes)
@@
 			)
 		)
-		(property "Footprint" ""
+		(property "Footprint" "Resistor_SMD:R_0805_2012Metric"
 			(at 226.822 55.88 90)
 			(hide yes)
@@
 		(in_pos_files yes)
 		(dnp no)
-		(fields_autoplaced yes)
 		(property "Reference" "Q1"
-			(at 242.57 43.18 0)
+			(at 238.76 46.99 0)
 			(show_name no)
 			(do_not_autoplace no)
@@
 		)
 		(property "Value" "IRLML2502"
-			(at 242.57 45.72 0)
+			(at 246.38 52.07 90)
 			(show_name no)
 			(do_not_autoplace no)
@@
 			)
 		)
-		(property "Datasheet" "https://www.infineon.com/dgdl/irlml2502pbf.pdf"
+		(property "Datasheet" "https://www.infineon.com/assets/row/public/documents/24/49/infineon-irlml2502-datasheet-en.pdf"
 			(at 242.57 50.8 0)
 			(hide yes)
@@
 			)
 		)
-		(property "Footprint" ""
+		(property "Footprint" "Resistor_SMD:R_0805_2012Metric"
 			(at 226.822 96.52 90)
 			(hide yes)
@@
 	(symbol
 		(lib_id "power:GND")
-		(at 250.19 58.42 0)
+		(at 242.57 55.88 0)
 		(unit 1)
 		(body_style 1)
@@
 		(fields_autoplaced yes)
 		(property "Reference" "#PWR042"
-			(at 250.19 64.77 0)
+			(at 242.57 62.23 0)
 			(hide yes)
 			(show_name no)
@@
 		)
 		(property "Value" "GND"
-			(at 250.19 63.5 0)
+			(at 242.57 60.96 0)
 			(show_name no)
 			(do_not_autoplace no)
@@
 		)
 		(property "Footprint" ""
-			(at 250.19 58.42 0)
+			(at 242.57 55.88 0)
 			(hide yes)
 			(show_name no)
@@
 		)
 		(property "Datasheet" ""
-			(at 250.19 58.42 0)
+			(at 242.57 55.88 0)
 			(hide yes)
 			(show_name no)
@@
 		)
 		(property "Description" "Power symbol creates a global label with name \"GND\" , ground"
-			(at 250.19 58.42 0)
+			(at 242.57 55.88 0)
 			(hide yes)
 			(show_name no)
@@
 			)
 		)
-		(property "Footprint" ""
+		(property "Footprint" "Resistor_SMD:R_0805_2012Metric"
 			(at 217.17 52.578 90)
 			(hide yes)
@@
 			)
 		)
-		(property "Footprint" ""
+		(property "Footprint" "Resistor_SMD:R_0805_2012Metric"
 			(at 218.44 91.948 90)
 			(hide yes)
