File: PCB/Center_Console/Center_Armament/AWRS_Panel/Controls.kicad_sch (KiCad schematic)
At the start: 0 parts

Commit message: chore: ignore .claire/ and .vscode/ dirs; save AWRS_Panel schematic state
- Expand .gitignore: add .claire/ (Claude Code worktrees), consolidate
  scattered .vscode/ file rules into a single **/.vscode/ glob
- AWRS_Panel.kicad_sch / Controls.kicad_sch: KiCad expanded embedded
  lib_symbols on open/save (Device:C_Small etc.)
- AWRS_Panel.kicad_pro: used_designators reset by KiCad on save
Parts:
- added R1, R10, R11, R12, R13, R2, R3, R4, R5, R6, R7, R8, R9: 1k, symbol Device:R_Small
- added SW1: SW_Rotary_1x12, symbol Switch:SW_Rotary_1x12
Connections:
- new net: R4.2, R5.1, SW1.4
- new net: R5.2, R6.1, SW1.5
- new net: R6.2, R7.1, SW1.6
- new net: R3.2, R4.1, SW1.3
- new net: R8.2, R9.1, SW1.8
- new net: R10.1, R9.2, SW1.9
- new net: R11.2, R12.1, SW1.11
- new net: R12.2, R13.1, SW1.12
- new net: R1.2, R2.1, SW1.1
- new net: R2.2, R3.1, SW1.2
- new net: R7.2, R8.1, SW1.7
- new net: R10.2, R11.1, SW1.10
- new net +3.3V: R1.1
- new net GND: R13.2
