File: PCB/Base/PanelGroup_Base/PanelGroup_Base.kicad_sch (KiCad schematic)
At the start: 0 parts

Commit message: feat(pcb): complete PanelGroup base board + CI fixes
PanelGroup_Base: schematic (ERC clean) + PCB layout (DRC clean).
Generic STM32F103C8 CAN sub-node - I2C with INT lines (8-pin),
backlight MOSFET drivers (Q2/Q3, PWM_BL1/BL2 on PA6/PA7), 2x7
breakout, 4x M2.5 mounting holes. Built by copy-paste from the
Gateway/Bridge base block. Prototype ordered from JLCPCB (red).

Gateway/Bridge: layout refinements (still ERC 0 / DRC 0).

Docs: base-boards.md backlight section synced to schematic naming
(PWM_BL1/BL2, BLn_RETURN, J_BL pin order). Added combined order BOM
CSV (both boards, deduped, for the LCSC order).

CI fixes:
- .gitattributes: mark 3D-model assets (*.STEP etc.) binary so
  `git diff --check` (PR Hygiene) skips their trailing whitespace.
- kicad-ci.yml: run the kicad-cli container as the runner UID with a
  writable HOME and mounted RUNNER_TEMP, fixing the
  "Directory '/home/runner' couldn't be created" DRC crash.

Both base boards verified ERC 0 / DRC 0. Pre-existing prototype ERC
failures (Armament_MCU, AWRS_Panel) are tracked as a separate task;
strict all-projects KiCad CI is intentionally kept, so this branch
stays red until those are fixed. Do not merge until then.
Parts:
- added C1: 100nf, Capacitor_SMD:C_0805_2012Metric, symbol Device:C
- added C10: 1uF, Capacitor_SMD:C_0805_2012Metric, symbol Device:C
- added C11: 10uF, Capacitor_SMD:CP_Elec_4x5.4, symbol Device:C_Polarized
- added C12, C2, C3, C4, C5, C6, C9: 100nF, Capacitor_SMD:C_0805_2012Metric, symbol Device:C
- added C13: 22uF, Capacitor_SMD:CP_Elec_4x5.4, symbol Device:C_Polarized
- added C14, C15: 10uF, Capacitor_SMD:C_0805_2012Metric, symbol Device:C
- added C7, C8: 22pF, Capacitor_SMD:C_0805_2012Metric, symbol Device:C
- added D1, D5: GREEN, LED_SMD:LED_0805_2012Metric, symbol Device:LED
- added D4: RED, LED_SMD:LED_0805_2012Metric, symbol Device:LED
- added H1, H2, H3, H4: MountingHole, MountingHole:MountingHole_2.7mm_M2.5, symbol Mechanical:MountingHole
- added J1: J_DIAG, Connector_JST:JST_XH_B3B-XH-A_1x03_P2.50mm_Vertical, symbol Connector_Generic:Conn_01x03
- added J11: J_BREAKOUT, Connector_PinHeader_2.54mm:PinHeader_2x07_P2.54mm_Vertical, symbol Connector_Generic:Conn_02x07_Odd_Even
- added J2: J_BL1, Connector_Molex:Molex_Mini-Fit_Jr_5566-02A_2x01_P4.20mm_Vertical, symbol Connector_Generic:Conn_01x02
- added J3: J_I2C2, Connector_JST:JST_XH_B8B-XH-A_1x08_P2.50mm_Vertical, symbol Connector_Generic:Conn_01x08
- added J4: J_I2C1, Connector_JST:JST_XH_B8B-XH-A_1x08_P2.50mm_Vertical, symbol Connector_Generic:Conn_01x08
- added J5: J_CAN_TERM, Connector_PinHeader_2.54mm:PinHeader_1x02_P2.54mm_Vertical, symbol Connector_Generic:Conn_01x02
- added J6: J_BL2, Connector_Molex:Molex_Mini-Fit_Jr_5566-02A_2x01_P4.20mm_Vertical, symbol Connector_Generic:Conn_01x02
- added J7: J_SWD, Connector_PinHeader_2.54mm:PinHeader_1x05_P2.54mm_Vertical, symbol Connector_Generic:Conn_01x05
- added J8: J_BUS_IN, Connector_Molex:Molex_Mini-Fit_Jr_5566-08A_2x04_P4.20mm_Vertical, symbol Connector_Generic:Conn_02x04_Top_Bottom
- added J9: J_BUS_OUT, Connector_Molex:Molex_Mini-Fit_Jr_5566-08A_2x04_P4.20mm_Vertical, symbol Connector_Generic:Conn_02x04_Top_Bottom
- added Q2, Q3: IRLML2502, Package_TO_SOT_SMD:SOT-23, symbol OpenSkyhawk:IRLML2502
- added R1, R10, R9: 3.3k, Resistor_SMD:R_0805_2012Metric, symbol Device:R
- added R11, R12, R18, R21, R22: 33, Resistor_SMD:R_0805_2012Metric, symbol Device:R
- added R13: 120, Resistor_SMD:R_0805_2012Metric, symbol Device:R
- added R16, R17, R19, R20, R23, R25: 100, Resistor_SMD:R_0805_2012Metric, symbol Device:R
- added R2, R3, R4, R5: 4.7k, Resistor_SMD:R_0805_2012Metric, symbol Device:R
- added R24, R26: 100k, Resistor_SMD:R_0805_2012Metric, symbol Device:R
- added R6: 10k, Resistor_SMD:R_0805_2012Metric, symbol Device:R
- added R_BOOT1: 10K, Resistor_SMD:R_0805_2012Metric, symbol Device:R
- added SW1: RESET, Button_Switch_THT:SW_PUSH_6mm, symbol Switch:SW_Push
- added U1: STM32F103C8Tx, Package_QFP:LQFP-48_7x7mm_P0.5mm, symbol MCU_ST_STM32F1:STM32F103C8Tx
- added U2: SN65HVD230, Package_SO:SOIC-8_3.9x4.9mm_P1.27mm, symbol Interface_CAN_LIN:SN65HVD230
- added U3: AMS1117-3.3, Package_TO_SOT_SMD:SOT-223-3_TabPin2, symbol Regulator_Linear:AMS1117-3.3
- added Y1: 8MHz, Crystal:Crystal_SMD_5032-2Pin_5.0x3.2mm, symbol Device:Crystal
Connections:
- new net: J3.7 (Pin_7), R17.2
- new net: J3.1 (Pin_1), R12.2
- new net: J3.2 (Pin_2), R11.1
- new net: J3.6 (Pin_6), R16.2
- new net: Q2.1, R23.2, R24.1
- new net: Q3.1, R25.2, R26.1
- new net: D1.1 (K), R1.1
- new net: J7.2 (Pin_2), R18.2
- new net: J5.1 (Pin_1), R13.2
- new net: D4.1 (K), R9.1
- new net: J4.6 (Pin_6), R19.2
- new net: J4.1 (Pin_1), R22.2
- new net: J4.2 (Pin_2), R21.1
- new net: J4.7 (Pin_7), R20.2
- new net: D5.1 (K), R10.1
- new net: R_BOOT1.1, U1.44 (BOOT0)
- new net +12V: C15.1, J2.1 (Pin_1), J6.1 (Pin_1), J8.1 (Pin_1), J8.2 (Pin_2), J9.1 (Pin_1), J9.2 (Pin_2)
- new net +3.3V: C1.1, C10.1, C12.1, C13.1, C2.1, C3.1, C4.1, C6.1, C9.1, D1.2 (A), J11.1 (Pin_1), J11.2 (Pin_2), J3.5 (Pin_5), J4.5 (Pin_5), J7.1 (Pin_1), R2.2, R3.1, R4.2, R5.1, R6.2, U1.1 (VBAT), U1.24 (VDD), U1.36 (VDD), U1.48 (VDD), U1.9 (VDDA), U2.3 (VCC), U3.2 (VO)
- new net +5V: C11.1, C14.1, J8.3 (Pin_3), J9.3 (Pin_3), U3.3 (VI)
- new net BL1_RETURN: J2.2 (Pin_2), Q2.3
- new net BL2_RETURN: J6.2 (Pin_2), Q3.3
- new net CANH: J8.5 (Pin_5), J9.5 (Pin_5), R13.1, U2.7 (CANH)
- new net CANL: J5.2 (Pin_2), J8.6 (Pin_6), J9.6 (Pin_6), U2.6 (CANL)
- new net CAN_RX: U1.32 (PA11), U2.4 (R)
- new net CAN_TX: U1.33 (PA12), U2.1 (D)
- new net DIAG_RX: J1.1 (Pin_1), U1.31 (PA10)
- new net DIAG_TX: J1.2 (Pin_2), U1.30 (PA9)
- new net GND: C1.2, C10.2, C11.2, C12.2, C13.2, C14.2, C15.2, C2.2, C3.2, C4.2, C5.2, C6.2, C7.1, C8.2, C9.2, J1.3 (Pin_3), J11.13 (Pin_13), J11.14 (Pin_14), J3.3 (Pin_3), J3.4 (Pin_4), J4.3 (Pin_3), J4.4 (Pin_4), J7.5 (Pin_5), J8.4 (Pin_4), J8.7 (Pin_7), J8.8 (Pin_8), J9.4 (Pin_4), J9.7 (Pin_7), J9.8 (Pin_8), Q2.2, Q3.2, R1.2, R10.2, R24.2, R26.2, R9.2, R_BOOT1.2, SW1.1, U1.23 (VSS), U1.35 (VSS), U1.47 (VSS), U1.8 (VSSA), U2.2 (GND), U2.8 (Rs), U3.1 (GND)
- new net I2C1_SCL: R2.1, R21.2, U1.42 (PB6)
- new net I2C1_SDA: R22.1, R4.1, U1.43 (PB7)
- new net I2C2_SCL: R11.2, R3.2, U1.21 (PB10)
- new net I2C2_SDA: R12.1, R5.2, U1.22 (PB11)
- new net INT_A1: R19.1, U1.25 (PB12)
- new net INT_A2: R16.1, U1.45 (PB8)
- new net INT_B1: R20.1, U1.26 (PB13)
- new net INT_B2: R17.1, U1.46 (PB9)
- new net NRST: C5.1, J7.4 (Pin_4), R6.1, SW1.2, U1.7 (NRST)
- new net OSC_IN: C8.1, U1.5 (PD0), Y1.2
- new net OSC_OUT: C7.2, U1.6 (PD1), Y1.1
- new net PA0: J11.4 (Pin_4), U1.10 (PA0)
- new net PA1: J11.6 (Pin_6), U1.11 (PA1)
- new net PA2: J11.8 (Pin_8), U1.12 (PA2)
- new net PA3: J11.10 (Pin_10), U1.13 (PA3)
- new net PA4: J11.12 (Pin_12), U1.14 (PA4)
- new net PA5: J11.9 (Pin_9), U1.15 (PA5)
- new net PA8: J11.11 (Pin_11), U1.29 (PA8)
- new net PANEL_GREEN: D5.2 (A), U1.28 (PB15)
- new net PANEL_RED: D4.2 (A), U1.27 (PB14)
- new net PB0: J11.3 (Pin_3), U1.18 (PB0)
- new net PB1: J11.5 (Pin_5), U1.19 (PB1)
- new net PB5: J11.7 (Pin_7), U1.41 (PB5)
- new net PWM_BL1: R23.1, U1.16 (PA6)
- new net PWM_BL2: R25.1, U1.17 (PA7)
- new net SWDCLK: J7.3 (Pin_3), U1.37 (PA14)
- new net SWDIO: R18.1, U1.34 (PA13)
- no-connect marks 0 -> 10
Other:
- note added: "CAN Bus"
- note added: "CAN Bus In"
- note added: "CAN Bus Out"
- note added: "PanelGroup MCU"
- note added: "PanelGroup Status"
- note added: "Power"
- note added: "Power Regulation"
- note added: "Programming"
- note added: "Status LED Indicators"
