File: PCB/Base/PanelGroup_Base/PanelGroup_Base.kicad_sch (KiCad schematic)
At the start: 64 parts, among them J1 J_DIAG, J11 J_BREAKOUT, J2 J_BL1, J3 J_I2C2, J4 J_I2C1, J5 J_CAN_TERM, J6 J_BL2, J7 J_SWD, J8 J_BUS_IN, J9 J_BUS_OUT, Q2 AO3400A, Q3 AO3400A, SW1 RESET, U1 STM32F103C8Tx, U2 SN65HVD230, U3 AMS1117-3.3, Y1 8MHz

Commit message: feat(pcb): label LCSC/tolerance/voltage across fleet boards (Right_Nav + PDU + base) (#235)
Populates **LCSC part number + tolerance + voltage** fields across all
six fleet boards, so each schematic drives an orderable BOM.

## Boards labeled (ERC 0/0 on all)
- **Right_Nav:** ASN-41, ARC-51A, APN-153
- **Power:** PDU
- **Base:** Gateway_Bridge, PanelGroup_Base

## What it does
- LCSC + tolerance + voltage on every assembled part, corrected to the
selected part (100nF 50V, resistors 1%, AMS1117 C6186→C347222, 10µF
split 25V/35V by +12V rail).
- Off-board panel controls (encoders, rotary switches, OLED, pot,
stepper, MEM button) left blank — connector-coupled, no assembly LCSC.
- Pin headers hand-soldered; RP2040-Zero left blank (module, sourced
separately).

## Design corrections captured here
- **PDU 1k series/anti-alias → 1%** (C110774 0.1% → C844939): precision
belongs only on the divider ratio resistors (33k/13k/10k); the series 1k
sit into high-Z ADC pins where 1% is identical. Drops the precision part
from the board.
- **DESIGN-NOTES:** records the 1k downgrade + the order-time shunt
upgrade (C346481 ±100ppm → C500740 ±25ppm, drop-in 2512).

## Not in this PR (follow-ups)
- Fleet component **standardization** (10µF-bulk→electrolytic,
consolidate to single 35V value, IPN convention) — separate pass.
- InvenTree backfill of the new SKUs.
Parts:
- C1: value 100nf -> 100nF; LCSC (none) -> C1711; Rating (none) -> 50V; Tolerance (none) -> 10%
- C10: LCSC (none) -> C28323; Rating (none) -> 50V; Tolerance (none) -> 10%
- C11: LCSC (none) -> C3343; Rating (none) -> 25V; Tolerance (none) -> 20%
- C12, C2, C3, C4, C5, C6, C9: LCSC (none) -> C1711; Rating (none) -> 50V; Tolerance (none) -> 10%
- C13: LCSC (none) -> C72502; Rating (none) -> 16V; Tolerance (none) -> 20%
- C14: value 10uF -> 100nF; LCSC (none) -> C1711; Rating (none) -> 50V; Tolerance (none) -> 10%
- C15: Rating (none) -> 35V; Tolerance (none) -> 20%
- C7, C8: LCSC (none) -> C1804; Rating (none) -> 50V; Tolerance (none) -> 5%
- D1, D5: LCSC (none) -> C19171393
- D3: Check_prices https://www.snapeda.com/parts/SMBJ5.0A/taiwan/view-part/?re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 -> (none); MF Taiwan Semiconductor -> MSKSEMI; PARTREV F2102 -> NA; Package SMD-2 Taiwan Semiconductor -> SMD-2; Purchase-URL https://www.snapeda.com/api/url_track_click_mouser/?unipart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 -> https://www.lcsc.com/product-detail/TVS_Diodes_MSKSEMI_SMBJ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; SnapEDA_Link https://www.snapeda.com/parts/SMBJ5.0A/taiwan/view-part/?re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 -> (none)
- D4: LCSC (none) -> C19171391
- J1: LCSC (none) -> C51940188
- J2, J6: LCSC (none) -> C20608113
- J3, J4: LCSC (none) -> C23067548
- J8, J9: LCSC (none) -> C20608116
- Q2, Q3: Rating (none) -> 30V
- R1, R10, R9: LCSC (none) -> C844412; Rating (none) -> 1/8W; Tolerance (none) -> 1%
- R11, R12, R18, R21, R22: LCSC (none) -> C2090807; Rating (none) -> 1/8W; Tolerance (none) -> 1%
- R13: LCSC (none) -> C844816; Rating (none) -> 1/8W; Tolerance (none) -> 1%
- R16, R17, R19, R20, R23, R25: LCSC (none) -> C844936; Rating (none) -> 1/8W; Tolerance (none) -> 1%
- R2, R3, R4, R5: LCSC (none) -> C844941; Rating (none) -> 1/8W; Tolerance (none) -> 1%
- R24, R26: LCSC (none) -> C844935; Rating (none) -> 1/8W; Tolerance (none) -> 1%
- R6: LCSC (none) -> C844937; Rating (none) -> 1/8W; Tolerance (none) -> 1%
- R_BOOT1: value 10K -> 10k; LCSC (none) -> C844937; Rating (none) -> 1/8W; Tolerance (none) -> 1%
- SW1: LCSC (none) -> C2939600
- U1: LCSC (none) -> C8734
- U2: LCSC (none) -> C12084
- U3: LCSC (none) -> C347222
- Y1: LCSC (none) -> C20617997
