File: PCB/Base/PanelGroup_Base/PanelGroup_Base.kicad_pcb (KiCad board)
At the start: 2 copper layers, 98 x 78.5 mm, 63 parts, among them J1 J_DIAG, J11 J_BREAKOUT, J2 J_BL1, J3 J_I2C2, J4 J_I2C1, J5 J_CAN_TERM, J6 J_BL2, J7 J_SWD, J8 J_BUS_IN, J9 J_BUS_OUT, Q2 IRLML2502, Q3 IRLML2502, SW1 RESET, U1 STM32F103C8Tx, U2 SN65HVD230, U3 AMS1117-3.3, Y1 8MHz

Commit message: feat(pcb): input-rail TVS + AO3400A backlight FET + 35V bus cap on base boards
Roll the #214 input-rail TVS fleet standard into both base boards, plus
two margin upgrades folded into the same rev:

- Input-rail TVS at J_BUS_IN on both boards: SMBJ12A (+12V, C42368008)
  and SMBJ6.0A (+5V, C5331096), cathode->rail / anode->GND, 2-3 GND
  vias at each anode pad for a low-inductance clamp path. CAN-bus TVS
  intentionally excluded (SN65HVD230 has built-in +/-16kV HBM).
- Backlight FET IRLML2502 -> AO3400A (C49195711, PanelGroup only):
  30V Vds vs 20V for headroom over the 19.9V clamp; Vgs operational at
  2.5V so still 3.3V-driven.
- +12V bulk cap C15 25V -> 35V X5R (C49010152): DC-bias derating +
  clamp headroom. C14 (+5V) stays 25V.

LCSC/MP/Voltage carried in-symbol. Combined BOM CSV + InvenTree updated.
DRC/ERC clean on both boards.

Refs #214
Parts:
- added D2: SMBJ12A, OpenSkyhawk:DIOM4336X265N, F.Cu at (133.5, 79.5)
- added D3: SMBJ6.0A, OpenSkyhawk:DIOM4336X265N, F.Cu at (119.8, 123.5)
- Q2, Q3: value IRLML2502 -> AO3400A
- moved C5 10.4 mm to (110.6, 129.5)
- moved R6 5.00 mm to (114.9, 129.4)
- moved SW1 0.46 mm to (108.8, 121.9)
Routing:
- net GND: track 91.7 -> 67.1 mm, vias 79 -> 86
- net +12V: track 86.9 -> 94.3 mm
- net +5V: track 11.6 -> 16.6 mm
- net +3.3V: track 360.3 -> 364.7 mm
- net /NRST: track 99.5 -> 98.3 mm, vias 4 -> 3

Commit message: feat(pcb): +12V bulk cap → 22µF/35V electrolytic reroute (#236) (#243)
## What
Replaces the **+12V bulk cap** across ASN-41, PDU, Gateway_Bridge and
PanelGroup_Base:
**10µF/35V ceramic (0805) → 22µF/35V aluminium electrolytic**
`C48971029` (`Capacitor_SMD:CP_Elec_5x5.4`).

## Why (#236)
- 10µF/35V *ceramic* on a 12V rail DC-bias-derates to ~4–6µF;
electrolytic holds full value at ~1/5 the cost.
- Footprint grows 0805 → Ø5 (35V elec), so fabbed boards get a reroute;
value taken to 22µF (same Ø5 can) for margin.

## Changes
- Symbol fields updated: IPN `CAP-ELEC-22UF-35V-D5`, LCSC `C48971029`,
Rating `35V`, Tolerance `20%`.
- **PDU (C9), Gateway_Bridge (C15), PanelGroup_Base (C15)** — rerouted
for the Ø5 land; board revision **0.1.0 → 0.2.0**.
- **ASN-41 (C15)** — unrouted, schematic only; revision **0.1.0**.

## Verification
- ERC clean (0/0) on all four boards.
- CI (KiCad PR Reports) runs ERC/DRC.

Closes #236 — the +12V ceramic→electrolytic reroute was the
consolidation's last open action; the rest is decided and applied (per
#235 + this PR).
Parts:
- C1: value 100nf -> 100nF
- C14: value 10uF -> 100nF
- C15: value 10uF -> 22uF; footprint Capacitor_SMD:C_0805_2012Metric -> Capacitor_SMD:CP_Elec_5x5.4
- R_BOOT1: value 10K -> 10k
- moved C15 30.3 mm to (122.9, 77.7), turned to 90 degrees
Routing:
- net GND: track 67.1 -> 63.7 mm

Commit message: feat(pcb): base boards Rev 2 — PanelGroup ShiftBus remap + Gateway/PDU fab prep (#209) (#302)
Takes PanelGroup base to Rev 2 for the 74HC ShiftBus pin standard, and
prepares
Gateway_Bridge and PDU for the same fab run. Boards are ordered — JLC
`W2026093021050394`, LCSC `WM2610010130` — so this is the as-fabricated
state.

## PanelGroup base Rev 2 (#209)

- **`J_SR` ShiftBus connector** (XH-7): `SCK · MOSI · MISO · GND · 3.3V
· LOAD · LTCH`,
  with 33 Ω series termination at the driver on SCK / LOAD / LATCH.
- **Nine-pin re-map.** I²C2 interrupts move PB8/PB9 → PA8/PA15 to free
the ShiftBus
strobes; J11 positions 7 and 11 become PB2 and PC14. PB2/PC14 are chosen
so the
breakout never collides with the I²C interrupt EXTI lines, which are
shared by pin
  number across ports.
- Docs rewritten from the final netlist: `docs/_source/base-boards.md`,
plus the
  INT-pin guidance and the now-adopted `J_SR` standard.

All four Rev 1 pre-order bench checks passed, so no finding forced a Rev
2 change —
CAN at 502 kbps with ACK from a second node, I²C pull-ups and both buses
end to end,
backlight PWM at 1.000 kHz with the gate pull-downs holding through
reset. Results are
recorded in #209.

## Gateway_Bridge and PDU — fab prep

Both boards had diverged from their fabbed revision (#243 moved the +12
V bulk cap to a
22 µF/35 V electrolytic, and Gateway gained the input-rail TVS with **no
pads on the old
board**), and neither had been assembled — so both were re-fabbed rather
than built as-is.

The silkscreen gate caught three real defects on Gateway before fab:

- revision text still read `0.1.0`
- **J8/J9 (`J_BUS_IN`/`J_BUS_OUT`) had no pin labels at all** — 12 V and
CAN on two
  identical unkeyed Mini-Fit connectors side by side
- **J1 (`J_DIAG`, the serial console) was labelled `SDA`/`SCL`** instead
of `RX`/`TX`

Also fixed a `CAN TERM` legend implemented by overriding the footprint
`Value` field,
which raised a parity error and would have been silently erased by the
next schema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
Parts:
- added J10: J_SR, Connector_JST:JST_XH_B7B-XH-A_1x07_P2.50mm_Vertical, F.Cu at (192.5, 102.8)
- added R27: 33, Resistor_SMD:R_0805_2012Metric, F.Cu at (185.7, 94.6)
- added R28: 33, Resistor_SMD:R_0805_2012Metric, F.Cu at (185.7, 97.2)
- added R29: 33, Resistor_SMD:R_0805_2012Metric, F.Cu at (185.7, 92.1)
- moved J11 15.5 mm to (191.0, 112.4)
Connections:
- J11 pad 11: /PA8 -> /PC14
- J11 pad 7: /PB5 -> /PB2
- U1 pad 20: unconnected-(U1-PB2-Pad20) -> /PB2
- U1 pad 29: /PA8 -> /INT_A2
- U1 pad 3: unconnected-(U1-PC14-Pad3) -> /PC14
- U1 pad 38: unconnected-(U1-PA15-Pad38) -> /INT_B2
- U1 pad 39: unconnected-(U1-PB3-Pad39) -> /SR_SCK
- U1 pad 40: unconnected-(U1-PB4-Pad40) -> /SR_MISO
- U1 pad 41: /PB5 -> /SR_MOSI
- U1 pad 45: /INT_A2 -> /SR_LOAD
- U1 pad 46: /INT_B2 -> /SR_LATCH
Routing:
- net /SR_MISO: track 0.00 -> 62.6 mm, vias 0 -> 3
- net /PC14: track 0.00 -> 55.2 mm, vias 0 -> 3
- net /PA8: track 44.7 -> 0.00 mm, vias 3 -> 0
- net /SR_LATCH: track 0.00 -> 37.5 mm, vias 0 -> 6
- net /PB2: track 0.00 -> 35.7 mm, vias 0 -> 3
- net /PB5: track 35.0 -> 0.00 mm, vias 3 -> 0
- net /SR_MOSI: track 0.00 -> 31.3 mm, vias 0 -> 3
- net /SR_LOAD: track 0.00 -> 26.3 mm, vias 0 -> 4
- net +3.3V: track 364.7 -> 386.2 mm
- net /SR_SCK: track 0.00 -> 20.3 mm, vias 0 -> 4
- net /PB0: track 56.7 -> 43.2 mm, vias 1 -> 2
- net /PB1: track 53.5 -> 41.7 mm
- net Net-(J10-Pin_1): track 0.00 -> 9.44 mm
- net Net-(J10-Pin_6): track 0.00 -> 7.71 mm
- net Net-(J10-Pin_7): track 0.00 -> 7.70 mm
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Other:
- board text added: "INT.A"
- board text added: "INT.B"
- board text added: "LOAD"
- board text added: "LTCH"
- board text added: "MISO"
- board text added: "MOSI"
- board text added: "PB2"
- board text added: "PC14"
- board text added: "REVISION 0.2.0 | PANEL GROUP BREAKOUT BOARD"
- board text added: "SCK"
- board text added: "SCL"
- board text added: "SDA"
- board text removed: "PA8"
- board text removed: "PB5"
- board text removed: "REVISION 0.1.0 | PANEL GROUP BREAKOUT BOARD"
