File: PCB/Right_Console/Right_Navigation/APN-153_Doppler/APN-153_Doppler.kicad_sch (KiCad schematic)
At the start: 33 parts, among them J1 J_MCU, J2 J_DOPPLER_SEL, J3 J_MEM_BUTTON, J4 J_BACKLIGHT, Q1 2N7002, SW1 DOPPLER_SEL, U1 MCP23017x-x-SS, U2 DRV8833PWP, U3 ER_OLEDM0.91_1x-I2C

Commit message: fix(APN-153): MEM LED series R 220->100 ohm (~13mA, R16-503 yellow) (#229)
MEM pushbutton LED (R16-503, yellow) series resistor **220→100Ω** → ~13
mA on the existing +5V / 2N7002 low-side path.

Bench-characterized against the R16-503 (the lamp has an internal
current-limiting resistor):
- 5V + 220Ω → ~6 mA (dim)
- 5V resistor-less → ~23 mA (at LED max, too hot for continuous)
- **5V + 100Ω → ~13 mA** — matches the 3.3V-direct brightness,
comfortable margin under the ~20 mA rating.

One-value change, no other edits. Bench detail logged on #170.

refs #181
Parts:
- R15: value 220 -> 100
Changed lines of the file:
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@@
 			)
 		)
-		(property "Value" "220"
+		(property "Value" "100"
 			(at 172.7873 139.087 90)
 			(show_name no)

Commit message: feat(pcb): ASN-41_NavComputer B2 schematic — Right_Nav host board (#230)
B2 schematic for the **AN/ASN-41 Navigation Computer** — the host board
for the **Right_Navigation** controller (NODE 2, STM32F103C8T6). Carries
the MCU, both I²C buses, the 74HC165 ShiftBus, host ADC, and the
inter-board harnesses to APN-153 + ARC-51.

## Board
- **MCU core** — STM32F103C8 (CAN, USART1 diag, SWD, 8 MHz OSC, status
LED).
- **74HC165 ShiftBus** (SPI1-remap PB3=SCK/PB4=MISO, PB8=LOAD) — ASN's 7
REL encoders + switch inputs; chain terminates on-board (host-local, no
J_SR leaves the board). `SHIFTBUS_ISR_HZ=1000`.
- **Dual I²C** — I²C1 (PB6/7) → APN-153 leg; I²C2 (PB10/11) → ARC-51 +
the OLED display muxes. 4.7 k pull-ups per bus.
- **OLED mux** — host TCA9548A @0x70 (7 ASN readout OLEDs, all 0x3C
behind mux).
- **Host ADC** — PA0 = ARC MODE ladder, PA1 = VOL, each with a 1 kΩ +
100 nF RC filter at the pin.
- **Interrupts** — APN INT_A1 (PB12); ARC INT_A2 (PA8).
- **Backlight** — 2 PWM low-side zones (PA6/PA7).
- Harness connectors defined on the root sheet (J_I2C1 → APN,
J_ARC51A_I2C → ARC, J_BL_*, CAN in/out).

## Sign-off
Netlist-audit review (export → parse → check nets) caught + fixed: I²C2
SDA/SCL crossed at the mux; ARC INT sharing PB13 with no pull-up → moved
to its own PA8.

**ERC: clean — 0 errors, 0 warnings.**

Closes #177. Refs #168 (controller), #174 (host board folds into ASN-41
B2).
Connections:
- net +5V: now also J4.4 (Pin_4)
- net 12V_BACKLIGHT: no longer J4.4 (Pin_4)
Changed lines of the file:
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@@
 		)
 	)
-	(label "12V_BACKLIGHT"
-		(at 172.72 111.76 0)
-		(effects
-			(font
-				(size 1.27 1.27)
-			)
-			(justify left bottom)
-		)
-	)
 	(label "INT_B"
 		(at 63.5 53.34 180)
@@
 					(unit 1)
 				)
+			)
+		)
+	)
+	(symbol
+		(lib_id "power:+5V")
+		(at 172.72 111.76 270)
+		(unit 1)
+		(body_style 1)
+		(exclude_from_sim no)
+		(in_bom yes)
+		(on_board yes)
+		(in_pos_files yes)
+		(dnp no)
+		(fields_autoplaced yes)
+		(property "Reference" "#PWR023"
+			(at 168.91 111.76 0)
+			(hide yes)
+			(show_name no)
+			(do_not_autoplace no)
+			(effects
+				(font
+					(size 1.27 1.27)
+				)
+			)
+		)
+		(property "Value" "+5V"
+			(at 176.53 111.7599 90)
+			(show_name no)
+			(do_not_autoplace no)
+			(effects
+				(font
+					(size 1.27 1.27)
+				)
+				(justify left)
+			)
+		)
+		(property "Footprint" ""
+			(at 172.72 111.76 0)
+			(hide yes)
+			(show_name no)
+			(do_not_autoplace no)
+			(effects
+				(font
+					(size 1.27 1.27)
+				)
+			)
+		)
+		(property "Datasheet" ""
+			(at 172.72 111.76 0)
+			(hide yes)
+			(show_name no)
+			(do_not_autoplace no)
+			(effects
+				(font
+					(size 1.27 1.27)
+				)
+			)
+		)
+		(property "Description" "Power symbol creates a global label with name \"+5V\""
+			(at 172.72 111.76 0)
+			(hide yes)
+			(show_name no)
+			(do_not_autoplace no)
+			(effects
+				(font
+					(size 1.27 1.27)
+				)
+			)
+		)
+		(pin "1"
+		)
+		(instances
+			(project "APN-153_Doppler"
+				(path "/b6290b15-680a-4921-8d70-c618bdfe22af"
+					(reference "#PWR023")
+					(unit 1)
+				)

Commit message: feat(pcb): label LCSC/tolerance/voltage across fleet boards (Right_Nav + PDU + base) (#235)
Populates **LCSC part number + tolerance + voltage** fields across all
six fleet boards, so each schematic drives an orderable BOM.

## Boards labeled (ERC 0/0 on all)
- **Right_Nav:** ASN-41, ARC-51A, APN-153
- **Power:** PDU
- **Base:** Gateway_Bridge, PanelGroup_Base

## What it does
- LCSC + tolerance + voltage on every assembled part, corrected to the
selected part (100nF 50V, resistors 1%, AMS1117 C6186→C347222, 10µF
split 25V/35V by +12V rail).
- Off-board panel controls (encoders, rotary switches, OLED, pot,
stepper, MEM button) left blank — connector-coupled, no assembly LCSC.
- Pin headers hand-soldered; RP2040-Zero left blank (module, sourced
separately).

## Design corrections captured here
- **PDU 1k series/anti-alias → 1%** (C110774 0.1% → C844939): precision
belongs only on the divider ratio resistors (33k/13k/10k); the series 1k
sit into high-Z ADC pins where 1% is identical. Drops the precision part
from the board.
- **DESIGN-NOTES:** records the 1k downgrade + the order-time shunt
upgrade (C346481 ±100ppm → C500740 ±25ppm, drop-in 2512).

## Not in this PR (follow-ups)
- Fleet component **standardization** (10µF-bulk→electrolytic,
consolidate to single 35V value, IPN convention) — separate pass.
- InvenTree backfill of the new SKUs.
Parts:
- C1, C3, C7: footprint (none) -> Capacitor_SMD:C_0805_2012Metric; LCSC (none) -> C1711; Rating (none) -> 50V; Tolerance (none) -> 10%
- C2: value 10uF -> 1uF; footprint (none) -> Capacitor_SMD:C_0805_2012Metric; LCSC (none) -> C28323; Rating (none) -> 50V; Tolerance (none) -> 10%
- C4: footprint (none) -> Capacitor_SMD:C_0805_2012Metric; LCSC (none) -> C49010152; Rating (none) -> 35V; Tolerance (none) -> 20%
- C5: footprint (none) -> Capacitor_SMD:C_0805_2012Metric; LCSC (none) -> C87994; Rating (none) -> 25V; Tolerance (none) -> 10%
- C6: footprint (none) -> Capacitor_SMD:C_0805_2012Metric; LCSC (none) -> C1710; Rating (none) -> 50V; Tolerance (none) -> 10%
- D1, D2: footprint (none) -> OpenSkyhawk:LED_5050_Red
- J1: footprint (none) -> Connector_JST:JST_XH_B8B-XH-A_1x08_P2.50mm_Vertical; LCSC (none) -> C23067548
- J2: footprint (none) -> Connector_JST:JST_XH_B6B-XH-A_1x06_P2.50mm_Vertical; LCSC (none) -> C23067546
- J4: footprint (none) -> Connector_Molex:Molex_Mini-Fit_Jr_5566-04A2_2x02_P4.20mm_Vertical; LCSC (none) -> C20608114
- Q1: LCSC (none) -> C8545; Rating (none) -> 60V
- R1, R2: footprint (none) -> Resistor_SMD:R_0805_2012Metric; LCSC (none) -> C2090807; Rating (none) -> 1/8W; Tolerance (none) -> 1%
- R10, R11, R12, R5, R6, R7, R8, R9: value 10K -> 10k; footprint (none) -> Resistor_SMD:R_0805_2012Metric; LCSC (none) -> C844937; Rating (none) -> 1/8W; Tolerance (none) -> 1%
- R14: value 100K -> 100k; footprint (none) -> Resistor_SMD:R_0805_2012Metric; LCSC (none) -> C844935; Rating (none) -> 1/8W; Tolerance (none) -> 1%
- R15, R3, R4: footprint (none) -> Resistor_SMD:R_0805_2012Metric; LCSC (none) -> C844936; Rating (none) -> 1/8W; Tolerance (none) -> 1%
- U1: LCSC (none) -> C506653
- U2: LCSC (none) -> C50506

Commit message: feat(pcb): add descriptive IPN field to all on-board symbols (#238 Phase 3) (#239)
Phase 3 of the IPN convention (#238): adds a stable, descriptive
**Internal Part Number** to every on-board symbol, co-equal with LCSC.
BOMs now anchor on a fixed identity; the LCSC can change with
availability without altering the part's identity.

## What changed
- **352 symbols** across all 6 boards (multi-sheet aware) get an `IPN`
field. **51 distinct IPNs.** ERC clean fleet-wide.
- **Off-board controls** (encoders/switches/pots/OLED/stepper — no
footprint, connector-coupled) get **no IPN**, per the standing off-board
exclusion. On-board modules (RP2040-ZERO) and the RESET tact switch
**do** get IPNs.
- `.gitignore`: FreeCAD backups (`*.FCBak`/`*.FCStd1`) + KiCad ERC/DRC
reports (`*-erc.rpt`/`*-drc.rpt`).

## Scheme (descriptive, locked in #238)
`RES-10K-1PCT-0805` · `CAP-CER-100NF-50V-0805` · `CAP-ELEC-22UF-16V-D4`
· `IC-STM32F103C8-LQFP` · `CONN-XH-8P` · `TVS-SMBJ12A-SMB` ·
`FUSE-HOLDER-BLADE-DIP4` · `SW-TACT-6MM` · `MOD-RP2040-ZERO`.

Resolved the 3 open encoding items: ferrite → `FB-600R-0805` (TDK
600Ω@100MHz), NTC → `NTC-10K-1206` (APV 10K), fuse holder (C19727305 is
a *holder*, not a fuse) → one `FUSE-HOLDER-BLADE-DIP4`.

## Not in this PR (later phases of #238)
- **Phase 2 — InvenTree:** set the IPN field + link SupplierParts incl
backorder alternates (one IPN → many LCSC). This is what actually
delivers the churn-proofing; needs reviewed InvenTree writes.
- **Phase 4 — order flow:** resolve IPN → in-stock LCSC at order time.

Refs #238.
Parts:
- C1, C3, C7: IPN (none) -> CAP-CER-100NF-50V-0805
- C2: IPN (none) -> CAP-CER-1UF-50V-0805
- C4: IPN (none) -> CAP-CER-10UF-35V-0805
- C5: IPN (none) -> CAP-CER-2P2UF-25V-0805
- C6: IPN (none) -> CAP-CER-10NF-50V-0805
- J1: IPN (none) -> CONN-XH-8P
- J2: IPN (none) -> CONN-XH-6P
- J4: IPN (none) -> CONN-MF-4P
- Q1: IPN (none) -> Q-2N7002-SOT23
- R1, R2: IPN (none) -> RES-33R-1PCT-0805
- R10, R11, R12, R5, R6, R7, R8, R9: IPN (none) -> RES-10K-1PCT-0805
- R14: IPN (none) -> RES-100K-1PCT-0805
- R15, R3, R4: IPN (none) -> RES-100R-1PCT-0805
- U1: IPN (none) -> IC-MCP23017-SSOP
- U2: IPN (none) -> IC-DRV8833-SSOP
