File: PCB/System/OpenSkyhawk_System/OpenSkyhawk_System.kicad_sch (KiCad schematic)
At the start: 0 parts

Commit message: docs(system): Right_Nav interconnect + console drill-down sheets (WIP)
System-architecture drill-down: root + console sub-sheets (Left/Center/Right/
SimGateway) and Right_Navigation_PG interconnect. Right_Nav blocks relabeled
ASN-41 (HOST) / APN-153 / ARC-51; host buses stubbed (I2C-1/I2C-2/SPI-1).

Wiring intentionally deferred: host->sub-panel backend (MCP23017/I2C vs
74HC165+595/SPI) is undecided pending the bench spike (#197) -> #168 tabled.
Parts:
- added POWER_SUPPLY: ATX-24, symbol Connector:ATX-24
Connections:
- new net: POWER_SUPPLY.1 (+3.3V), POWER_SUPPLY.12 (+3.3V), POWER_SUPPLY.13 (+3.3V), POWER_SUPPLY.2 (+3.3V)
- new net GND: POWER_SUPPLY.15 (GND), POWER_SUPPLY.17 (GND), POWER_SUPPLY.18 (GND), POWER_SUPPLY.19 (GND), POWER_SUPPLY.24 (GND), POWER_SUPPLY.3 (GND), POWER_SUPPLY.5 (GND), POWER_SUPPLY.7 (GND)
- new net LEFT_CONSOLE/12V_IN: POWER_SUPPLY.10 (+12V), POWER_SUPPLY.11 (+12V)
- new net LEFT_CONSOLE/5V_IN: POWER_SUPPLY.21 (+5V), POWER_SUPPLY.22 (+5V), POWER_SUPPLY.23 (+5V), POWER_SUPPLY.4 (+5V), POWER_SUPPLY.6 (+5V)
- no-connect marks 0 -> 12
Other:
- added sheet Center_Console (Center_Console.kicad_sch)
- added sheet LEFT_CONSOLE (LEFT_CONSOLE.kicad_sch)
- added sheet Right Console (Right_Console.kicad_sch)
- added sheet SimGateway (SimGateway.kicad_sch)
- note added: "CAN BUS TERMINATION"
