File: PCB/Right_Console/Right_Navigation/ASN-41_NavComputer/Backlight.kicad_sch (KiCad schematic)
At the start: 8 parts, among them J7 J_BACKLIGHT, J8 J_ARC53_PANEL_BL, Q1 AO3400A, Q2 AO3400A

Commit message: chore(pcb): ASN-41 BOM fields + value-case/J8/C-rating fixes
Add LCSC/Tolerance/Rating/Notes fields to all components. Merge value-case (100nf->100nF, 10k->10K). Fix J8 label ARC53->ARC51. C13/C15 12V bulk -> 35V (SMBJ12A clamp margin, C49010152). Off-board notes on panel-mount switches.

refs #177
Parts:
- J8: value J_ARC53_PANEL_BL -> J_ARC51_PANEL_BL
- R48, R49, R50, R51: Rating (none) -> 1/8W; Tolerance (none) -> 5%
