File: PCB/Right_Console/Right_Navigation/ASN-41_NavComputer/MCU.kicad_sch (KiCad schematic)
At the start: 62 parts, among them J1 J_DIAG, J2 J_SWD, J3 J_BUS_IN, J4 J_CAN_TERM, J5 J_BUS_OUT, J6 J_APN153_I2C, J9 J_ARC51A_I2C, SW1 RESET, U1 STM32F103C8Tx, U2 AMS1117-3.3, U3 SN65HVD230, Y1 8MHz

Commit message: chore(pcb): ASN-41 BOM fields + value-case/J8/C-rating fixes
Add LCSC/Tolerance/Rating/Notes fields to all components. Merge value-case (100nf->100nF, 10k->10K). Fix J8 label ARC53->ARC51. C13/C15 12V bulk -> 35V (SMBJ12A clamp margin, C49010152). Off-board notes on panel-mount switches.

refs #177
Parts:
- C1, C28, C29: value 100nf -> 100nF; Rating (none) -> 16V; Tolerance (none) -> 10%
- C10, C11, C12, C14, C2, C3, C4, C5, C6, C7: Rating (none) -> 16V; Tolerance (none) -> 10%
- C13: Rating (none) -> 35V; Tolerance (none) -> 10%
- C15: Notes (none) -> 35V min — SMBJ12A clamp ~20V; Rating (none) -> 35V; Tolerance (none) -> 10%
- C8, C9: Notes (none) -> C0G/NP0; Rating (none) -> 50V; Tolerance (none) -> 5%
- R1, R10, R11, R12, R13, R14, R2, R3, R4, R5, R52, R54, R55, R7, R8, R9, R_BOOT1: Rating (none) -> 1/8W; Tolerance (none) -> 5%
- R53, R56: Rating (none) -> 1/8W; Tolerance (none) -> 1%
- R6: value 10k -> 10K; Rating (none) -> 1/8W; Tolerance (none) -> 5%
- U1: LCSC (none) -> C8734
- U2: LCSC (none) -> C6186
- U3: LCSC (none) -> C12084
