File: PCB/Right_Console/Right_Navigation/ASN-41_NavComputer/MCU.kicad_sch (KiCad schematic)
At the start: 62 parts, among them J1 J_DIAG, J2 J_SWD, J3 J_BUS_IN, J4 J_CAN_TERM, J5 J_BUS_OUT, J6 J_APN153_I2C, J9 J_ARC51A_I2C, SW1 RESET, U1 STM32F103C8Tx, U2 AMS1117-3.3, U3 SN65HVD230, Y1 8MHz

Commit message: feat(pcb): label LCSC/tolerance/voltage across fleet boards (Right_Nav + PDU + base) (#235)
Populates **LCSC part number + tolerance + voltage** fields across all
six fleet boards, so each schematic drives an orderable BOM.

## Boards labeled (ERC 0/0 on all)
- **Right_Nav:** ASN-41, ARC-51A, APN-153
- **Power:** PDU
- **Base:** Gateway_Bridge, PanelGroup_Base

## What it does
- LCSC + tolerance + voltage on every assembled part, corrected to the
selected part (100nF 50V, resistors 1%, AMS1117 C6186→C347222, 10µF
split 25V/35V by +12V rail).
- Off-board panel controls (encoders, rotary switches, OLED, pot,
stepper, MEM button) left blank — connector-coupled, no assembly LCSC.
- Pin headers hand-soldered; RP2040-Zero left blank (module, sourced
separately).

## Design corrections captured here
- **PDU 1k series/anti-alias → 1%** (C110774 0.1% → C844939): precision
belongs only on the divider ratio resistors (33k/13k/10k); the series 1k
sit into high-Z ADC pins where 1% is identical. Drops the precision part
from the board.
- **DESIGN-NOTES:** records the 1k downgrade + the order-time shunt
upgrade (C346481 ±100ppm → C500740 ±25ppm, drop-in 2512).

## Not in this PR (follow-ups)
- Fleet component **standardization** (10µF-bulk→electrolytic,
consolidate to single 35V value, IPN convention) — separate pass.
- InvenTree backfill of the new SKUs.
Parts:
- C1, C10, C14, C2, C28, C29, C3, C4, C5, C6: LCSC (none) -> C1711; Rating 16V -> 50V
- C11: LCSC (none) -> C28323; Rating 16V -> 50V
- C12: LCSC (none) -> C72502; Tolerance 10% -> 20%
- C13: value 10uF -> 100nF; LCSC (none) -> C1711; Rating 35V -> 50V
- C15: Tolerance 10% -> 20%
- C7: LCSC (none) -> C3343; Rating 16V -> 25V; Tolerance 10% -> 20%
- C8, C9: LCSC (none) -> C1804
- D1, D3: LCSC (none) -> C19171393
- D2: LCSC (none) -> C19171391
- J1: LCSC (none) -> C51940188
- J3, J5: LCSC (none) -> C20608116
- J6, J9: LCSC (none) -> C23067548
- R1, R7, R8: LCSC (none) -> C844412; Tolerance 5% -> 1%
- R10: LCSC (none) -> C844816; Tolerance 5% -> 1%
- R11, R12, R52: LCSC (none) -> C844936; Tolerance 5% -> 1%
- R13, R14, R54, R55, R9: LCSC (none) -> C2090807; Tolerance 5% -> 1%
- R2, R3, R4, R5: LCSC (none) -> C844941; Tolerance 5% -> 1%
- R53, R56: value 1K -> 1k; LCSC (none) -> C844939
- R6, R_BOOT1: value 10K -> 10k; LCSC (none) -> C844937; Tolerance 5% -> 1%
- SW1: LCSC (none) -> C2939600
- U2: LCSC C6186 -> C347222
- Y1: LCSC (none) -> C20617997
