File: PCB/Right_Console/Right_Navigation/ASN-41_NavComputer/MCU.kicad_sch (KiCad schematic)
At the start: 62 parts, among them J1 J_DIAG, J2 J_SWD, J3 J_BUS_IN, J4 J_CAN_TERM, J5 J_BUS_OUT, J6 J_APN153_I2C, J9 J_ARC51A_I2C, SW1 RESET, U1 STM32F103C8Tx, U2 AMS1117-3.3, U3 SN65HVD230, Y1 8MHz

Commit message: feat(pcb): label LCSC/tolerance/voltage on Right_Nav + PDU schematics
Populate LCSC, Tolerance, and Rating (voltage/power) fields across the four
fabbed boards, sourced from InvenTree + the board tickets and PDU DESIGN-NOTES.
Values corrected to the selected part (100nF 50V, resistors 1%, AMS1117
C6186 -> C347222, 10uF split 25V/35V by +12V rail).

- PDU: dividers 0.1% (C2828767/C865184/C406725/C110774), J1 Mini-Fit 4-pin
  C20608114, D3/D4 green, C9 35V on +12V (SMBJ12A clamp margin).
- ARC-51A: MCP23017 C506653, TCA9548 C130026, J9 XH-8 C23067548, backlight
  J8 Mini-Fit 2-pin C20608113.
- ASN-41: AMS1117 C347222, TCA9548 C130026, 10uF per-rail split, 74HC165 x4
  C22384789, 1k ADC filter C844939, backlight J8 C20608113.
- APN-153: footprints (0805 passives + XH/Mini-Fit connectors) + MCP23017
  C506653, DRV8833 C50506, 2N7002 C8545, 2.2uF C87994 (25V X5R), 10nF C1710,
  6-pin XH J2 C23067546.

Off-board panel controls (encoders, rotary switches, OLED, pot, stepper, MEM
button) excluded as connector-coupled. Pin headers (SWD, CAN_TERM) hand-
soldered, no assembly LCSC. Harness mating ends tracked in the order BOM.
Parts:
- C1, C10, C14, C2, C28, C29, C3, C4, C5, C6: LCSC (none) -> C1711; Rating 16V -> 50V
- C11: LCSC (none) -> C28323; Rating 16V -> 50V
- C12: LCSC (none) -> C72502; Tolerance 10% -> 20%
- C13: LCSC (none) -> C669099; Rating 35V -> 25V; Tolerance 10% -> 20%
- C15: Tolerance 10% -> 20%
- C7: LCSC (none) -> C3343; Rating 16V -> 25V; Tolerance 10% -> 20%
- C8, C9: LCSC (none) -> C1804
- D1, D3: LCSC (none) -> C19171393
- D2: LCSC (none) -> C19171391
- J1: LCSC (none) -> C51940188
- J3, J5: LCSC (none) -> C20608116
- J6, J9: LCSC (none) -> C23067548
- R1, R7, R8: LCSC (none) -> C844412; Tolerance 5% -> 1%
- R10: LCSC (none) -> C844816; Tolerance 5% -> 1%
- R11, R12, R52: LCSC (none) -> C844936; Tolerance 5% -> 1%
- R13, R14, R54, R55, R9: LCSC (none) -> C2090807; Tolerance 5% -> 1%
- R2, R3, R4, R5: LCSC (none) -> C844941; Tolerance 5% -> 1%
- R53, R56: LCSC (none) -> C844939
- R6, R_BOOT1: LCSC (none) -> C844937; Tolerance 5% -> 1%
- SW1: LCSC (none) -> C2939600
- U2: LCSC C6186 -> C347222
- Y1: LCSC (none) -> C20617997

Commit message: chore(pcb): normalize passive value-string case fleet-wide
Cosmetic cleanup — standardize resistor/cap value strings so identical
parts stop showing as separate BOM lines. Value = magnitude only;
tolerance + LCSC carry the precision distinction.

- 10K -> 10k, 4.7K -> 4.7k, 100K -> 100k (lowercase SI k)
- 100nf -> 100nF
- 69 symbols across all 6 boards (ASN-41, ARC-51A, APN-153, PDU,
  Gateway_Bridge, PanelGroup_Base). ERC 0/0 on all.

No functional/footprint/LCSC change. PDU generic 10k and precision
divider 10k now both read "10k", distinguished by tolerance (1% vs 0.1%).
Parts:
- R6, R_BOOT1: value 10K -> 10k
Changed lines of the file:
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@@
 			)
 		)
-		(property "Value" "10K"
+		(property "Value" "10k"
 			(at 33.02 139.7 90)
 			(show_name no)
@@
 			)
 		)
-		(property "Value" "10K"
+		(property "Value" "10k"
 			(at 22.86 60.96 0)
 			(show_name no)

Commit message: chore(pcb): normalize remaining uppercase-K resistor values
Completes the value-string cleanup — the first pass only caught the
case-duplicate values (10K/4.7K/100K). This fixes the uppercase-K values
that had no lowercase twin: 1K, 1.5K, 13K, 33K -> lowercase k.

13 symbols. All 6 boards now fully SI-consistent (lowercase k, uppercase
F); zero remaining violations, ERC 0/0.
Parts:
- R53, R56: value 1K -> 1k
Changed lines of the file:
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@@
 			)
 		)
-		(property "Value" "1K"
+		(property "Value" "1k"
 			(at 242.57 91.44 90)
 			(show_name no)
@@
 			)
 		)
-		(property "Value" "1K"
+		(property "Value" "1k"
 			(at 242.57 99.06 90)
 			(show_name no)

Commit message: refactor(pcb): consolidate ceramic 10uF to single 35V part
The 10uF ceramic 0805 caps were split across two SKUs — C669099 (25V)
and C49010152 (35V) — distinguished only by rail. Standardize all 8
ceramic positions to the 35V part (C49010152); 35V covers the 25V
positions and collapses the BOM to one ceramic 10uF value.

Electrolytic 10uF (C3343) unchanged. Aluminum-bulk replacement deferred
to a future round. 8 caps across all 6 boards, ERC 0/0.
Parts:
- C13: LCSC C669099 -> C49010152; Rating 25V -> 35V
Changed lines of the file:
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@@
 			)
 		)
-		(property "LCSC" "C669099"
+		(property "LCSC" "C49010152"
 			(at 0 0 0)
 			(hide yes)
@@
 			)
 		)
-		(property "Rating" "25V"
+		(property "Rating" "35V"
 			(at 0 0 0)
 			(hide yes)

Commit message: fix(pcb): re-value AMS1117 input ceramic 10uF->100nF (ASN/PDU/Gate/Pane)
The AMS1117 +5V input carried two bulk caps (10uF ceramic + 10uF elec)
and no HF bypass. Re-value the redundant 10uF ceramic to 100nF (reuse
C1711, 0805 unchanged) so each input = 10uF elec bulk + 100nF ceramic
HF = standard LDO input. No footprint/symbol change; ERC clean.
Frees another 10uF/35V ceramic and closes the missing-input-HF gap.
Parts:
- C13: value 10uF -> 100nF; LCSC C49010152 -> C1711; Rating 35V -> 50V; Tolerance 20% -> 10%
Changed lines of the file:
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@@
 			)
 		)
-		(property "Value" "10uF"
+		(property "Value" "100nF"
 			(at 134.62 38.0999 0)
 			(show_name no)
@@
 			)
 		)
-		(property "LCSC" "C49010152"
+		(property "LCSC" "C1711"
 			(at 0 0 0)
 			(hide yes)
@@
 			)
 		)
-		(property "Tolerance" "20%"
+		(property "Tolerance" "10%"
 			(at 0 0 0)
 			(hide yes)
@@
 			)
 		)
-		(property "Rating" "35V"
+		(property "Rating" "50V"
 			(at 0 0 0)
 			(hide yes)

Commit message: feat(pcb): add descriptive IPN field to all on-board symbols (#238 Phase 3) (#239)
Phase 3 of the IPN convention (#238): adds a stable, descriptive
**Internal Part Number** to every on-board symbol, co-equal with LCSC.
BOMs now anchor on a fixed identity; the LCSC can change with
availability without altering the part's identity.

## What changed
- **352 symbols** across all 6 boards (multi-sheet aware) get an `IPN`
field. **51 distinct IPNs.** ERC clean fleet-wide.
- **Off-board controls** (encoders/switches/pots/OLED/stepper — no
footprint, connector-coupled) get **no IPN**, per the standing off-board
exclusion. On-board modules (RP2040-ZERO) and the RESET tact switch
**do** get IPNs.
- `.gitignore`: FreeCAD backups (`*.FCBak`/`*.FCStd1`) + KiCad ERC/DRC
reports (`*-erc.rpt`/`*-drc.rpt`).

## Scheme (descriptive, locked in #238)
`RES-10K-1PCT-0805` · `CAP-CER-100NF-50V-0805` · `CAP-ELEC-22UF-16V-D4`
· `IC-STM32F103C8-LQFP` · `CONN-XH-8P` · `TVS-SMBJ12A-SMB` ·
`FUSE-HOLDER-BLADE-DIP4` · `SW-TACT-6MM` · `MOD-RP2040-ZERO`.

Resolved the 3 open encoding items: ferrite → `FB-600R-0805` (TDK
600Ω@100MHz), NTC → `NTC-10K-1206` (APV 10K), fuse holder (C19727305 is
a *holder*, not a fuse) → one `FUSE-HOLDER-BLADE-DIP4`.

## Not in this PR (later phases of #238)
- **Phase 2 — InvenTree:** set the IPN field + link SupplierParts incl
backorder alternates (one IPN → many LCSC). This is what actually
delivers the churn-proofing; needs reviewed InvenTree writes.
- **Phase 4 — order flow:** resolve IPN → in-stock LCSC at order time.

Refs #238.
Parts:
- C1, C10, C13, C14, C2, C28, C29, C3, C4, C5, C6: IPN (none) -> CAP-CER-100NF-50V-0805
- C11: IPN (none) -> CAP-CER-1UF-50V-0805
- C12: IPN (none) -> CAP-ELEC-22UF-16V-D4
- C15: IPN (none) -> CAP-CER-10UF-35V-0805
- C7: IPN (none) -> CAP-ELEC-10UF-25V-D4
- C8, C9: IPN (none) -> CAP-C0G-22PF-50V-0805
- D1, D3: IPN (none) -> LED-GREEN-0805
- D2: IPN (none) -> LED-RED-0805
- D4: IPN (none) -> TVS-SMBJ6V0A-SMB
- D5: IPN (none) -> TVS-SMBJ12A-SMB
- J1: IPN (none) -> CONN-XH-3P
- J2: IPN (none) -> CONN-HDR-5P
- J3, J5: IPN (none) -> CONN-MF-8P
- J4: IPN (none) -> CONN-HDR-2P
- J6, J9: IPN (none) -> CONN-XH-8P
- R1, R7, R8: IPN (none) -> RES-3K3-1PCT-0805
- R10: IPN (none) -> RES-120R-1PCT-0805
- R11, R12, R52: IPN (none) -> RES-100R-1PCT-0805
- R13, R14, R54, R55, R9: IPN (none) -> RES-33R-1PCT-0805
- R2, R3, R4, R5: IPN (none) -> RES-4K7-1PCT-0805
- R53, R56: IPN (none) -> RES-1K-1PCT-0805
- R6, R_BOOT1: IPN (none) -> RES-10K-1PCT-0805
- SW1: IPN (none) -> SW-TACT-6MM
- U1: IPN (none) -> IC-STM32F103C8-LQFP
- U2: IPN (none) -> IC-AMS1117-3V3-SOT223
- U3: IPN (none) -> IC-SN65HVD230-SOIC
- Y1: IPN (none) -> XTAL-8MHZ-SMD5032

Commit message: feat(pcb): +12V bulk cap → 22µF/35V electrolytic reroute (#236) (#243)
## What
Replaces the **+12V bulk cap** across ASN-41, PDU, Gateway_Bridge and
PanelGroup_Base:
**10µF/35V ceramic (0805) → 22µF/35V aluminium electrolytic**
`C48971029` (`Capacitor_SMD:CP_Elec_5x5.4`).

## Why (#236)
- 10µF/35V *ceramic* on a 12V rail DC-bias-derates to ~4–6µF;
electrolytic holds full value at ~1/5 the cost.
- Footprint grows 0805 → Ø5 (35V elec), so fabbed boards get a reroute;
value taken to 22µF (same Ø5 can) for margin.

## Changes
- Symbol fields updated: IPN `CAP-ELEC-22UF-35V-D5`, LCSC `C48971029`,
Rating `35V`, Tolerance `20%`.
- **PDU (C9), Gateway_Bridge (C15), PanelGroup_Base (C15)** — rerouted
for the Ø5 land; board revision **0.1.0 → 0.2.0**.
- **ASN-41 (C15)** — unrouted, schematic only; revision **0.1.0**.

## Verification
- ERC clean (0/0) on all four boards.
- CI (KiCad PR Reports) runs ERC/DRC.

Closes #236 — the +12V ceramic→electrolytic reroute was the
consolidation's last open action; the rest is decided and applied (per
#235 + this PR).
Parts:
- removed C15: 10uF, Capacitor_SMD:C_0805_2012Metric, symbol Device:C
- added C15: 22uF, Capacitor_SMD:CP_Elec_5x5.4, symbol Device:C_Polarized_Small
Connections:
- net +12V: now also C15.1
- net GND: now also C15.2
