File: PCB/Right_Console/Right_Navigation/ASN-41_NavComputer/Oled_Displays.kicad_sch (KiCad schematic)
At the start: 17 parts, among them U10 ER_OLEDM0.91_1x-I2C, U11 ER_OLEDM0.91_1x-I2C, U4 TCA9548APWR, U5 ER_OLEDM0.91_1x-I2C, U6 ER_OLEDM0.91_1x-I2C, U7 ER_OLEDM0.91_1x-I2C, U8 ER_OLEDM0.91_1x-I2C, U9 ER_OLEDM0.91_1x-I2C

Commit message: chore(pcb): ASN-41 BOM fields + value-case/J8/C-rating fixes
Add LCSC/Tolerance/Rating/Notes fields to all components. Merge value-case (100nf->100nF, 10k->10K). Fix J8 label ARC53->ARC51. C13/C15 12V bulk -> 35V (SMBJ12A clamp margin, C49010152). Off-board notes on panel-mount switches.

refs #177
Parts:
- C16, C17, C18, C19, C20, C21, C22, C23: Rating (none) -> 16V; Tolerance (none) -> 10%
- R15: Rating (none) -> 1/8W; Tolerance (none) -> 5%
- U10, U11, U5, U6, U7, U8, U9: Notes (none) -> OLED module, off-board mount
- U4: LCSC (none) -> C130026
