File: PCB/Right_Console/Right_Navigation/ASN-41_NavComputer/Switches.kicad_sch (KiCad schematic)
At the start: 52 parts, among them SW10 LONG_SLEW_W, SW11 LAT_SLEW_N, SW12 MAG_VAR, SW13 W_DIR, SW2 PP_LAT, SW3 PP_LONG, SW4 W_SPEED, SW5 LONG_SLEW_E, SW6 LAT_SLEW_S, SW7 DT_LAT, SW8 DT_LONG, SW9 NAV_SELECTOR, U12 74HC165, U13 74HC165, U14 74HC165, U15 74HC165

Commit message: chore(pcb): ASN-41 BOM fields + value-case/J8/C-rating fixes
Add LCSC/Tolerance/Rating/Notes fields to all components. Merge value-case (100nf->100nF, 10k->10K). Fix J8 label ARC53->ARC51. C13/C15 12V bulk -> 35V (SMBJ12A clamp margin, C49010152). Off-board notes on panel-mount switches.

refs #177
Parts:
- C24, C25, C26, C27: Rating (none) -> 16V; Tolerance (none) -> 10%
- R16, R17, R18, R19, R20, R21, R22, R23, R24, R25, R26, R27, R28, R29, R30, R31, R32, R33, R34, R35, R36, R37, R38, R39, R40, R41, R42, R43, R44, R45, R46, R47: Rating (none) -> 1/8W; Tolerance (none) -> 5%
- SW10, SW11, SW12, SW13, SW2, SW3, SW4, SW5, SW6, SW7, SW8, SW9: Notes (none) -> off-board — PCB-direct or JST-XH (decide at B5)
