File: PCB/Right_Console/Right_Navigation/ASN-41_NavComputer/Switches.kicad_sch (KiCad schematic)
At the start: 52 parts, among them SW10 LONG_SLEW_W, SW11 LAT_SLEW_N, SW12 MAG_VAR, SW13 W_DIR, SW2 PP_LAT, SW3 PP_LONG, SW4 W_SPEED, SW5 LONG_SLEW_E, SW6 LAT_SLEW_S, SW7 DT_LAT, SW8 DT_LONG, SW9 NAV_SELECTOR, U12 74HC165, U13 74HC165, U14 74HC165, U15 74HC165

Commit message: feat(pcb): label LCSC/tolerance/voltage on Right_Nav + PDU schematics
Populate LCSC, Tolerance, and Rating (voltage/power) fields across the four
fabbed boards, sourced from InvenTree + the board tickets and PDU DESIGN-NOTES.
Values corrected to the selected part (100nF 50V, resistors 1%, AMS1117
C6186 -> C347222, 10uF split 25V/35V by +12V rail).

- PDU: dividers 0.1% (C2828767/C865184/C406725/C110774), J1 Mini-Fit 4-pin
  C20608114, D3/D4 green, C9 35V on +12V (SMBJ12A clamp margin).
- ARC-51A: MCP23017 C506653, TCA9548 C130026, J9 XH-8 C23067548, backlight
  J8 Mini-Fit 2-pin C20608113.
- ASN-41: AMS1117 C347222, TCA9548 C130026, 10uF per-rail split, 74HC165 x4
  C22384789, 1k ADC filter C844939, backlight J8 C20608113.
- APN-153: footprints (0805 passives + XH/Mini-Fit connectors) + MCP23017
  C506653, DRV8833 C50506, 2N7002 C8545, 2.2uF C87994 (25V X5R), 10nF C1710,
  6-pin XH J2 C23067546.

Off-board panel controls (encoders, rotary switches, OLED, pot, stepper, MEM
button) excluded as connector-coupled. Pin headers (SWD, CAN_TERM) hand-
soldered, no assembly LCSC. Harness mating ends tracked in the order BOM.
Parts:
- C24, C25, C26, C27: LCSC (none) -> C1711; Rating 16V -> 50V
- R16, R17, R18, R19, R20, R21, R22, R23, R24, R25, R26, R27, R28, R29, R30, R31, R32, R33, R34, R35, R36, R37, R38, R39, R40, R41, R42, R43, R44, R45, R46, R47: LCSC (none) -> C844937; Tolerance 5% -> 1%
- U12, U13, U14, U15: LCSC (none) -> C22384789

Commit message: chore(pcb): normalize passive value-string case fleet-wide
Cosmetic cleanup — standardize resistor/cap value strings so identical
parts stop showing as separate BOM lines. Value = magnitude only;
tolerance + LCSC carry the precision distinction.

- 10K -> 10k, 4.7K -> 4.7k, 100K -> 100k (lowercase SI k)
- 100nf -> 100nF
- 69 symbols across all 6 boards (ASN-41, ARC-51A, APN-153, PDU,
  Gateway_Bridge, PanelGroup_Base). ERC 0/0 on all.

No functional/footprint/LCSC change. PDU generic 10k and precision
divider 10k now both read "10k", distinguished by tolerance (1% vs 0.1%).
Parts:
- R16, R17, R18, R19, R20, R21, R22, R23, R24, R25, R26, R27, R28, R29, R30, R31, R32, R33, R34, R35, R36, R37, R38, R39, R40, R41, R42, R43, R44, R45, R46, R47: value 10K -> 10k
Changed lines of the file:
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@@
 			)
 		)
-		(property "Value" "10K"
+		(property "Value" "10k"
 			(at 25.4 83.82 90)
 			(show_name no)
@@
 			)
 		)
-		(property "Value" "10K"
+		(property "Value" "10k"
 			(at 25.4 111.76 90)
 			(show_name no)
@@
 			)
 		)
-		(property "Value" "10K"
+		(property "Value" "10k"
 			(at 55.88 38.1 90)
 			(show_name no)
@@
 			)
 		)
-		(property "Value" "10K"
+		(property "Value" "10k"
 			(at 25.4 73.66 90)
 			(show_name no)
@@
 			)
 		)
-		(property "Value" "10K"
+		(property "Value" "10k"
 			(at 142.24 73.66 90)
 			(show_name no)
@@
 			)
 		)
-		(property "Value" "10K"
+		(property "Value" "10k"
 			(at 88.9 53.34 90)
 			(show_name no)
@@
 			)
 		)
-		(property "Value" "10K"
+		(property "Value" "10k"
 			(at 160.02 160.02 90)
 			(hide yes)
@@
 			)
 		)
-		(property "Value" "10K"
+		(property "Value" "10k"
 			(at 86.36 73.66 90)
 			(show_name no)
@@
 			)
 		)
-		(property "Value" "10K"
+		(property "Value" "10k"
 			(at 86.36 121.92 90)
 			(show_name no)
@@
 			)
 		)
-		(property "Value" "10K"
+		(property "Value" "10k"
 			(at 172.72 73.66 90)
 			(show_name no)
@@
 			)
 		)
-		(property "Value" "10K"
+		(property "Value" "10k"
 			(at 86.36 83.82 90)
 			(show_name no)
@@
 			)
 		)
-		(property "Value" "10K"
+		(property "Value" "10k"
 			(at 198.12 68.58 90)
 			(show_name no)
@@
 			)
 		)
-		(property "Value" "10K"
+		(property "Value" "10k"
 			(at 154.94 160.02 90)
 			(hide yes)
@@
 			)
 		)
-		(property "Value" "10K"
+		(property "Value" "10k"
 			(at 116.84 73.66 90)
 			(show_name no)
@@
 			)
 		)
-		(property "Value" "10K"
+		(property "Value" "10k"
 			(at 154.94 165.1 0)
 			(show_name no)
@@
 			)
 		)
-		(property "Value" "10K"
+		(property "Value" "10k"
 			(at 147.32 160.02 90)
 			(hide yes)
@@
 			)
 		)
-		(property "Value" "10K"
+		(property "Value" "10k"
 			(at 142.24 121.92 90)
 			(show_name no)
@@
 			)
 		)
-		(property "Value" "10K"
+		(property "Value" "10k"
 			(at 86.36 111.76 90)
 			(show_name no)
@@
 			)
 		)
-		(property "Value" "10K"
+		(property "Value" "10k"
 			(at 55.88 111.76 90)
 			(show_name no)
@@
 			)
 		)
-		(property "Value" "10K"
+		(property "Value" "10k"
 			(at 142.24 83.82 90)
 			(show_name no)
@@
 			)
 		)
-		(property "Value" "10K"
+		(property "Value" "10k"
 			(at 142.24 111.76 90)
 			(show_name no)
@@
 			)
 		)
-		(property "Value" "10K"
+		(property "Value" "10k"
 			(at 127 53.34 90)
 			(show_name no)
@@
 			)
 		)
-		(property "Value" "10K"
+		(property "Value" "10k"
 			(at 116.84 111.76 90)
 			(show_name no)
@@
 			)
 		)
-		(property "Value" "10K"
+		(property "Value" "10k"
 			(at 55.88 73.66 90)
 			(show_name no)
@@
 			)
 		)
-		(property "Value" "10K"
+		(property "Value" "10k"
 			(at 25.4 48.26 90)
 			(show_name no)
@@
 			)
 		)
-		(property "Value" "10K"
+		(property "Value" "10k"
 			(at 25.4 121.92 90)
 			(show_name no)
@@
 			)
 		)
-		(property "Value" "10K"
+		(property "Value" "10k"
 			(at 175.26 111.76 90)
 			(show_name no)
@@
 			)
 		)
-		(property "Value" "10K"
+		(property "Value" "10k"
 			(at 88.9 38.1 90)
 			(show_name no)
@@
 			)
 		)
-		(property "Value" "10K"
+		(property "Value" "10k"
 			(at 25.4 38.1 90)
 			(show_name no)
@@
 			)
 		)
-		(property "Value" "10K"
+		(property "Value" "10k"
 			(at 198.12 60.96 90)
 			(hide yes)
@@
 			)
 		)
-		(property "Value" "10K"
+		(property "Value" "10k"
 			(at 127 38.1 90)
 			(show_name no)
@@
 			)
 		)
-		(property "Value" "10K"
+		(property "Value" "10k"
 			(at 157.48 160.02 90)
 			(hide yes)
