File: PCB/Right_Console/Right_Navigation/ASN-41_NavComputer/Switches.kicad_sch (KiCad schematic)
At the start: 52 parts, among them SW10 LONG_SLEW_W, SW11 LAT_SLEW_N, SW12 MAG_VAR, SW13 W_DIR, SW2 PP_LAT, SW3 PP_LONG, SW4 W_SPEED, SW5 LONG_SLEW_E, SW6 LAT_SLEW_S, SW7 DT_LAT, SW8 DT_LONG, SW9 NAV_SELECTOR, U12 74HC165, U13 74HC165, U14 74HC165, U15 74HC165

Commit message: fix(pcb): Right_Nav harness-contract fixes — J7 5V, '165 spares, APN sync
Netlist-audit follow-ups on the ASN-41 host + APN-153 mate:
- J7 dual-zone backlight pin 4 -> +5V utility (standard dual-zone; was +12V)
- U12 '165 spare inputs D6/D7 (R46/R47) -> +3V3 pull-up (was GND) — matches
  the board's active-low scheme + all other inputs, restores wire-and-go
- APN-153: J4 backlight pin 4 -> +5V, aligning the mate to the host J7

Confirmed correct as-is (no change): J6/J1 I2C pin-8 +5V (trunk-sourced flex
for APN's 5V stepper/MEM) and J8 J_BL order (matches the fabbed PanelGroup_Base).
ERC: 0.
Connections:
- net +3.3V: now also R46.2, R47.2
- net GND: no longer R46.2, R47.2
Changed lines of the file:
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@@
 	)
 	(symbol
-		(lib_id "power:GND")
-		(at 193.04 66.04 270)
-		(unit 1)
-		(body_style 1)
-		(exclude_from_sim no)
-		(in_bom yes)
-		(on_board yes)
-		(in_pos_files yes)
-		(dnp no)
-		(property "Reference" "#PWR0107"
-			(at 186.69 66.04 0)
-			(hide yes)
-			(show_name no)
-			(do_not_autoplace no)
-			(effects
-				(font
-					(size 1.27 1.27)
-				)
-			)
-		)
-		(property "Value" "GND"
-			(at 189.702 65.9179 90)
-			(show_name no)
-			(do_not_autoplace no)
-			(effects
-				(font
-					(size 1.27 1.27)
-				)
-				(justify right)
-			)
-		)
-		(property "Footprint" ""
-			(at 193.04 66.04 0)
-			(hide yes)
-			(show_name no)
-			(do_not_autoplace no)
-			(effects
-				(font
-					(size 1.27 1.27)
-				)
-			)
-		)
-		(property "Datasheet" ""
-			(at 193.04 66.04 0)
-			(hide yes)
-			(show_name no)
-			(do_not_autoplace no)
-			(effects
-				(font
-					(size 1.27 1.27)
-				)
-			)
-		)
-		(property "Description" "Power symbol creates a global label with name \"GND\" , ground"
-			(at 193.04 66.04 0)
-			(hide yes)
-			(show_name no)
-			(do_not_autoplace no)
-			(effects
-				(font
-					(size 1.27 1.27)
-				)
-			)
-		)
-		(pin "1"
-		)
-		(instances
-			(project "ASN-41_NavComputer"
-				(path "/44380fee-2d92-4c15-902c-f5cfd680baf1/e80a81f1-1a88-4a6d-8836-9196b5a0533f"
-					(reference "#PWR0107")
-					(unit 1)
-				)
-			)
-		)
-	)
-	(symbol
 		(lib_id "Device:R_Small")
 		(at 25.4 114.3 90)
@@
 					(unit 1)
 				)
+			)
+		)
+	)
+	(symbol
+		(lib_id "power:+3.3V")
+		(at 193.04 66.04 90)
+		(unit 1)
+		(body_style 1)
+		(exclude_from_sim no)
+		(in_bom yes)
+		(on_board yes)
+		(in_pos_files yes)
+		(dnp no)
+		(fields_autoplaced yes)
+		(property "Reference" "#PWR0107"
+			(at 196.85 66.04 0)
+			(hide yes)
+			(show_name no)
+			(do_not_autoplace no)
+			(effects
+				(font
+					(size 1.27 1.27)
+				)
+			)
+		)
+		(property "Value" "+3.3V"
+			(at 189.23 66.0399 90)
+			(show_name no)
+			(do_not_autoplace no)
+			(effects
+				(font
+					(size 1.27 1.27)
+				)
+				(justify left)
+			)
+		)
+		(property "Footprint" ""
+			(at 193.04 66.04 0)
+			(hide yes)
+			(show_name no)
+			(do_not_autoplace no)
+			(effects
+				(font
+					(size 1.27 1.27)
+				)
+			)
+		)
+		(property "Datasheet" ""
+			(at 193.04 66.04 0)
+			(hide yes)
+			(show_name no)
+			(do_not_autoplace no)
+			(effects
+				(font
+					(size 1.27 1.27)
+				)
+			)
+		)
+		(property "Description" "Power symbol creates a global label with name \"+3.3V\""
+			(at 193.04 66.04 0)
+			(hide yes)
+			(show_name no)
+			(do_not_autoplace no)
+			(effects
+				(font
+					(size 1.27 1.27)
+				)
+			)
+		)
+		(pin "1"
+		)
+		(instances
+			(project "ASN-41_NavComputer"
+				(path "/44380fee-2d92-4c15-902c-f5cfd680baf1/e80a81f1-1a88-4a6d-8836-9196b5a0533f"
+					(reference "#PWR0107")
+					(unit 1)
+				)

Commit message: feat(pcb): label LCSC/tolerance/voltage across fleet boards (Right_Nav + PDU + base) (#235)
Populates **LCSC part number + tolerance + voltage** fields across all
six fleet boards, so each schematic drives an orderable BOM.

## Boards labeled (ERC 0/0 on all)
- **Right_Nav:** ASN-41, ARC-51A, APN-153
- **Power:** PDU
- **Base:** Gateway_Bridge, PanelGroup_Base

## What it does
- LCSC + tolerance + voltage on every assembled part, corrected to the
selected part (100nF 50V, resistors 1%, AMS1117 C6186→C347222, 10µF
split 25V/35V by +12V rail).
- Off-board panel controls (encoders, rotary switches, OLED, pot,
stepper, MEM button) left blank — connector-coupled, no assembly LCSC.
- Pin headers hand-soldered; RP2040-Zero left blank (module, sourced
separately).

## Design corrections captured here
- **PDU 1k series/anti-alias → 1%** (C110774 0.1% → C844939): precision
belongs only on the divider ratio resistors (33k/13k/10k); the series 1k
sit into high-Z ADC pins where 1% is identical. Drops the precision part
from the board.
- **DESIGN-NOTES:** records the 1k downgrade + the order-time shunt
upgrade (C346481 ±100ppm → C500740 ±25ppm, drop-in 2512).

## Not in this PR (follow-ups)
- Fleet component **standardization** (10µF-bulk→electrolytic,
consolidate to single 35V value, IPN convention) — separate pass.
- InvenTree backfill of the new SKUs.
Parts:
- C24, C25, C26, C27: LCSC (none) -> C1711; Rating 16V -> 50V
- R16, R17, R18, R19, R20, R21, R22, R23, R24, R25, R26, R27, R28, R29, R30, R31, R32, R33, R34, R35, R36, R37, R38, R39, R40, R41, R42, R43, R44, R45, R46, R47: value 10K -> 10k; LCSC (none) -> C844937; Tolerance 5% -> 1%
- U12, U13, U14, U15: LCSC (none) -> C22384789

Commit message: feat(pcb): add descriptive IPN field to all on-board symbols (#238 Phase 3) (#239)
Phase 3 of the IPN convention (#238): adds a stable, descriptive
**Internal Part Number** to every on-board symbol, co-equal with LCSC.
BOMs now anchor on a fixed identity; the LCSC can change with
availability without altering the part's identity.

## What changed
- **352 symbols** across all 6 boards (multi-sheet aware) get an `IPN`
field. **51 distinct IPNs.** ERC clean fleet-wide.
- **Off-board controls** (encoders/switches/pots/OLED/stepper — no
footprint, connector-coupled) get **no IPN**, per the standing off-board
exclusion. On-board modules (RP2040-ZERO) and the RESET tact switch
**do** get IPNs.
- `.gitignore`: FreeCAD backups (`*.FCBak`/`*.FCStd1`) + KiCad ERC/DRC
reports (`*-erc.rpt`/`*-drc.rpt`).

## Scheme (descriptive, locked in #238)
`RES-10K-1PCT-0805` · `CAP-CER-100NF-50V-0805` · `CAP-ELEC-22UF-16V-D4`
· `IC-STM32F103C8-LQFP` · `CONN-XH-8P` · `TVS-SMBJ12A-SMB` ·
`FUSE-HOLDER-BLADE-DIP4` · `SW-TACT-6MM` · `MOD-RP2040-ZERO`.

Resolved the 3 open encoding items: ferrite → `FB-600R-0805` (TDK
600Ω@100MHz), NTC → `NTC-10K-1206` (APV 10K), fuse holder (C19727305 is
a *holder*, not a fuse) → one `FUSE-HOLDER-BLADE-DIP4`.

## Not in this PR (later phases of #238)
- **Phase 2 — InvenTree:** set the IPN field + link SupplierParts incl
backorder alternates (one IPN → many LCSC). This is what actually
delivers the churn-proofing; needs reviewed InvenTree writes.
- **Phase 4 — order flow:** resolve IPN → in-stock LCSC at order time.

Refs #238.
Parts:
- C24, C25, C26, C27: IPN (none) -> CAP-CER-100NF-50V-0805
- R16, R17, R18, R19, R20, R21, R22, R23, R24, R25, R26, R27, R28, R29, R30, R31, R32, R33, R34, R35, R36, R37, R38, R39, R40, R41, R42, R43, R44, R45, R46, R47: IPN (none) -> RES-10K-1PCT-0805
- U12, U13, U14, U15: IPN (none) -> IC-74HC165-SOIC
