File: PCB/Base/Gateway_Bridge/Gateway_Bridge.kicad_sch (KiCad schematic)
At the start: 59 parts, among them J1 J_DIAG, J2 J_I2C2, J3 STM32_Breakout, J5 J_CAN_TERM, J6 J_I2C1, J7 J_SWD, J8 J_BUS_IN, J9 J_BUS_OUT, SW1 RESET, U1 STM32F103C8Tx, U2 SN65HVD230, U3 AMS1117-3.3, U4 RP2040-ZERO, Y1 8MHz

Commit message: feat(pcb): label base boards + PDU 1k downgrade to 1%
Extends the LCSC/tolerance/voltage labeling to the two base boards and
corrects a PDU over-spec.

- Gateway_Bridge, PanelGroup_Base: LCSC + tolerance + voltage on all
  parts (footprints already present). 10uF split 25V/35V by +12V rail.
  RP2040-Zero left blank (module, ordered separately, no LCSC); pin
  headers hand-soldered (no assembly LCSC).
- PDU: R8-R12/R15-R17 (1k series/anti-alias) downgraded C110774 0.1%
  -> C844939 1%. Precision belongs only on the divider ratio resistors
  (33k/13k/10k); the series 1k sit into high-Z ADC pins where 1% reads
  identically. Drops the precision C110774 from the board entirely.
- DESIGN-NOTES: record the 1k downgrade + the order-time shunt upgrade
  (C346481 100ppm -> C500740 25ppm).
Parts:
- C1, C12, C2, C3, C4, C5, C6, C9: LCSC (none) -> C1711; Rating (none) -> 50V; Tolerance (none) -> 10%
- C10: LCSC (none) -> C28323; Rating (none) -> 50V; Tolerance (none) -> 10%
- C11: LCSC (none) -> C3343; Rating (none) -> 25V; Tolerance (none) -> 20%
- C13: LCSC (none) -> C72502; Rating (none) -> 16V; Tolerance (none) -> 20%
- C14: LCSC (none) -> C669099; Rating (none) -> 25V; Tolerance (none) -> 20%
- C15: Rating (none) -> 35V; Tolerance (none) -> 20%
- C7, C8: LCSC (none) -> C1804; Rating (none) -> 50V; Tolerance (none) -> 5%
- D1, D3, D5: LCSC (none) -> C19171393
- D2, D4: LCSC (none) -> C19171391
- D7: LCSC (none) -> C42368008
- J1: LCSC (none) -> C51940188
- J2, J6: LCSC (none) -> C23067544
- J8, J9: LCSC (none) -> C20608116
- R1, R10, R7, R8, R9: LCSC (none) -> C844412; Rating (none) -> 1/8W; Tolerance (none) -> 1%
- R11, R12, R14, R15, R16, R17, R18: LCSC (none) -> C2090807; Rating (none) -> 1/8W; Tolerance (none) -> 1%
- R13: LCSC (none) -> C844816; Rating (none) -> 1/8W; Tolerance (none) -> 1%
- R2, R3, R4, R5: LCSC (none) -> C844941; Rating (none) -> 1/8W; Tolerance (none) -> 1%
- R6, R_BOOT1: LCSC (none) -> C844937; Rating (none) -> 1/8W; Tolerance (none) -> 1%
- SW1: LCSC (none) -> C2939600
- U1: LCSC (none) -> C8734
- U2: LCSC (none) -> C12084
- U3: LCSC (none) -> C347222
- Y1: LCSC (none) -> C20617997

Commit message: chore(pcb): normalize passive value-string case fleet-wide
Cosmetic cleanup — standardize resistor/cap value strings so identical
parts stop showing as separate BOM lines. Value = magnitude only;
tolerance + LCSC carry the precision distinction.

- 10K -> 10k, 4.7K -> 4.7k, 100K -> 100k (lowercase SI k)
- 100nf -> 100nF
- 69 symbols across all 6 boards (ASN-41, ARC-51A, APN-153, PDU,
  Gateway_Bridge, PanelGroup_Base). ERC 0/0 on all.

No functional/footprint/LCSC change. PDU generic 10k and precision
divider 10k now both read "10k", distinguished by tolerance (1% vs 0.1%).
Parts:
- C1: value 100nf -> 100nF
- R_BOOT1: value 10K -> 10k
Changed lines of the file:
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@@
 			)
 		)
-		(property "Value" "100nf"
+		(property "Value" "100nF"
 			(at 20.32 35.56 0)
 			(show_name no)
@@
 			)
 		)
-		(property "Value" "10K"
+		(property "Value" "10k"
 			(at 24.13 60.96 0)
 			(show_name no)
