File: PCB/Base/Gateway_Bridge/Gateway_Bridge.kicad_sch (KiCad schematic)
At the start: 59 parts, among them J1 J_DIAG, J2 J_I2C2, J3 STM32_Breakout, J5 J_CAN_TERM, J6 J_I2C1, J7 J_SWD, J8 J_BUS_IN, J9 J_BUS_OUT, SW1 RESET, U1 STM32F103C8Tx, U2 SN65HVD230, U3 AMS1117-3.3, U4 RP2040-ZERO, Y1 8MHz

Commit message: refactor(pcb): consolidate ceramic 10uF to single 35V part
The 10uF ceramic 0805 caps were split across two SKUs — C669099 (25V)
and C49010152 (35V) — distinguished only by rail. Standardize all 8
ceramic positions to the 35V part (C49010152); 35V covers the 25V
positions and collapses the BOM to one ceramic 10uF value.

Electrolytic 10uF (C3343) unchanged. Aluminum-bulk replacement deferred
to a future round. 8 caps across all 6 boards, ERC 0/0.
Parts:
- C14: LCSC C669099 -> C49010152; Rating 25V -> 35V
Changed lines of the file:
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@@
 			)
 		)
-		(property "Rating" "25V"
+		(property "Rating" "35V"
 			(at 218.44 36.83 0)
 			(hide yes)
@@
 			)
 		)
-		(property "LCSC" "C669099"
+		(property "LCSC" "C49010152"
 			(at 218.44 36.83 0)
 			(hide yes)

Commit message: fix(pcb): correct SMBJ6.0A TVS metadata on PDU/base boards
D2 (PDU), D6 (Gateway_Bridge), D3 (PanelGroup_Base) carried stale
SnapEDA metadata from the original SMBJ5.0A (Taiwan Semiconductor)
symbol after the value was swapped to the 6.0A part. Value + LCSC
(C5331096) were already correct; this aligns the rest so BOM/inventory
exports agree with InvenTree:
- MF Taiwan Semiconductor -> MSKSEMI (actual mfr of C5331096)
- MP SMBJ5.0A -> SMBJ6.0A (PDU; already correct on base boards)
- Description 5V -> 6V
- Purchase-URL -> LCSC product page; clear stale SnapEDA links,
  Taiwan-Semi PARTREV/Package refs

ERC clean on all three.
Parts:
- D6: Check_prices https://www.snapeda.com/parts/SMBJ5.0A/taiwan/view-part/?re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 -> (none); MF Taiwan Semiconductor -> MSKSEMI; PARTREV F2102 -> NA; Package SMD-2 Taiwan Semiconductor -> SMD-2; Purchase-URL https://www.snapeda.com/api/url_track_click_mouser/?unipart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 -> https://www.lcsc.com/product-detail/TVS_Diodes_MSKSEMI_SMBJ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; SnapEDA_Link https://www.snapeda.com/parts/SMBJ5.0A/taiwan/view-part/?re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 -> (none)
Changed lines of the file:
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@@
 			)
 		)
-		(property "Description" "600W, 5V, Unidirectional, TVS"
+		(property "Description" "600W, 6V, Unidirectional, TVS"
 			(at 209.55 36.83 0)
 			(hide yes)
@@
 			)
 		)
-		(property "MF" "Taiwan Semiconductor"
+		(property "MF" "MSKSEMI"
 			(at 209.55 36.83 0)
 			(hide yes)
@@
 			)
 		)
-		(property "Package" "SMD-2 Taiwan Semiconductor"
+		(property "Package" "SMD-2"
 			(at 209.55 36.83 0)
 			(hide yes)
@@
 			)
 		)
-		(property "Check_prices" "https://www.snapeda.com/parts/SMBJ5.0A/taiwan/view-part/?ref=eda"
+		(property "Check_prices" ""
 			(at 209.55 36.83 0)
 			(hide yes)
@@
 			)
 		)
-		(property "PARTREV" "F2102"
+		(property "PARTREV" "NA"
 			(at 209.55 36.83 0)
 			(hide yes)
@@
 			)
 		)
-		(property "SnapEDA_Link" "https://www.snapeda.com/parts/SMBJ5.0A/taiwan/view-part/?ref=snap"
+		(property "SnapEDA_Link" ""
 			(at 209.55 36.83 0)
 			(hide yes)
@@
 			)
 		)
-		(property "Purchase-URL" "https://www.snapeda.com/api/url_track_click_mouser/?unipart_id=1860032&manufacturer=Taiwan Semiconductor&part_name=SMBJ5.0A&search_term=smbj5.0a"
+		(property "Purchase-URL" "https://www.lcsc.com/product-detail/TVS_Diodes_MSKSEMI_SMBJ6.0A_C5331096.html"
 			(at 209.55 36.83 0)
 			(hide yes)

Commit message: fix(pcb): drop stray LCSV typo field on Gateway_Bridge D7
D7 (SMBJ12A) had a duplicate mislabeled "LCSV" property alongside the
correct LCSC=C42368008. Harmless to the BOM but pollutes field audits.
Removed; LCSC intact, ERC clean.
Parts:
- D7: LCSV C42368008 -> (none)
Changed lines of the file:
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@@
-			)
-		)
-		(property "LCSV" "C42368008"
-			(at 261.62 38.1 90)
-			(hide yes)
-			(show_name no)
-			(do_not_autoplace no)
-			(effects
-				(font
-					(size 1.27 1.27)
-				)
 			)
 		)

Commit message: fix(pcb): re-value AMS1117 input ceramic 10uF->100nF (ASN/PDU/Gate/Pane)
The AMS1117 +5V input carried two bulk caps (10uF ceramic + 10uF elec)
and no HF bypass. Re-value the redundant 10uF ceramic to 100nF (reuse
C1711, 0805 unchanged) so each input = 10uF elec bulk + 100nF ceramic
HF = standard LDO input. No footprint/symbol change; ERC clean.
Frees another 10uF/35V ceramic and closes the missing-input-HF gap.
Parts:
- C14: value 10uF -> 100nF; LCSC C49010152 -> C1711; Rating 35V -> 50V; Tolerance 20% -> 10%
Changed lines of the file:
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@@
 			)
 		)
-		(property "Value" "10uF"
+		(property "Value" "100nF"
 			(at 222.25 38.0999 0)
 			(show_name no)
@@
 			)
 		)
-		(property "Rating" "35V"
+		(property "Rating" "50V"
 			(at 218.44 36.83 0)
 			(hide yes)
@@
 			)
 		)
-		(property "Tolerance" "20%"
+		(property "Tolerance" "10%"
 			(at 218.44 36.83 0)
 			(hide yes)
@@
 			)
 		)
-		(property "LCSC" "C49010152"
+		(property "LCSC" "C1711"
 			(at 218.44 36.83 0)
 			(hide yes)
