File: PCB/Base/Gateway_Bridge/Gateway_Bridge.kicad_pcb (KiCad board)
At the start: 2 copper layers, 98.9 x 70.1 mm, 60 parts, among them J1 J_DIAG, J2 J_I2C2, J3 STM32_Breakout, J5 J_CAN_TERM, J6 J_I2C1, J7 J_SWD, J8 J_BUS_IN, J9 J_BUS_OUT, SW1 RESET, U1 STM32F103C8Tx, U2 SN65HVD230, U3 AMS1117-3.3, U4 RP2040-ZERO, Y1 8MHz

Commit message: fix(pcb): Gateway UART series resistors R16/R17 33 Ω → 1k (#356)
Parts:
- R16, R17: value 33 -> 1k
Other:
- board text added: "REVISION 0.2.1 | GATEWAY BRIDGE"
- board text removed: "REVISION 0.2.0 | GATEWAY BRIDGE"
Changed lines of the file:
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@@
 	)
 	(paper "A4")
+	(title_block
+		(title "Gateway_Bridge")
+		(date "2026-06-16")
+		(rev "0.2.1")
+		(company "OpenSkyhawk")
+	)
 	(layers
 		(0 "F.Cu" signal)
@@
 			)
 		)
-		(property "Value" "33"
+		(property "Value" "1k"
 			(at 0 1.65 0)
 			(layer "F.Fab")
@@
 			)
 		)
-		(property "IPN" "RES-33R-1PCT-0805"
+		(property "IPN" "RES-1K-1PCT-0805"
 			(at 0 0 0)
 			(unlocked yes)
@@
 			)
 		)
-		(property "LCSC" "C2090807"
+		(property "LCSC" "C844939"
 			(at 0 0 0)
 			(unlocked yes)
@@
 			)
 		)
-		(property "Value" "33"
+		(property "Value" "1k"
 			(at 0 1.65 0)
 			(layer "F.Fab")
@@
 			)
 		)
-		(property "IPN" "RES-33R-1PCT-0805"
+		(property "IPN" "RES-1K-1PCT-0805"
 			(at 0 0 0)
 			(unlocked yes)
@@
 			)
 		)
-		(property "LCSC" "C2090807"
+		(property "LCSC" "C844939"
 			(at 0 0 0)
 			(unlocked yes)
@@
 		)
 	)
-	(gr_text "REVISION 0.2.0 | GATEWAY BRIDGE"
+	(gr_text "REVISION 0.2.1 | GATEWAY BRIDGE"
 		(at 75.5 147.525 0)
 		(layer "B.SilkS")
