File: PCB/Base/Power/PDU/PDU.kicad_sch (KiCad schematic)
At the start: 0 parts

Commit message: feat(pcb): PDU schematic front-end — sensing, protection, MCU ADC (#202)
Draw the PDU-specific circuitry (standard STM32 block imported next
session):

- Input: Mini-Fit Jr 4-pin (12V/GND/GND/5V), input-rail TVS
  (SMBJ12A/SMBJ5.0A) shunt-to-GND, MINI-blade fuses (12V 5A / 5V 2A)
- Voltage sense: load-side dividers -> 12V_READ_ADC / 5V_READ_ADC
- Current sense: INA180A2 (gain 50) across 10mR shunts, RC-filtered
  outputs -> I_12V_ADC / I_5V_ADC
- Temp: 10k NTC divider -> NTC_ADC
- STM32: VDDA ferrite-bead filter, ADC map PA0-3 + PA6
- Power indicators: MCU-independent 12V/5V rail LEDs

DESIGN-NOTES: full BOM with LCSC part numbers, ADC map, CAN-node reuse
(STM32Board + CANProtocol), reserved pins, remaining steps.

Footprints + standard-block import + ERC deferred to next session.
Parts:
- added C1, C2, C3, C4, C5, C6, C7, C8: 100nF, symbol Device:C_Small
- added C9: 1uF, symbol Device:C_Small
- added D1: SMBJ5.0A, SMBJ5.0A:DIOM4336X265N, symbol OpenSkyhawk:SMBJ5.0A
- added D2: SMBJ12A, SMBJ12A:DIOM4336X265N, symbol OpenSkyhawk:SMBJ12A
- added D3: 12V_ST, symbol Device:LED_Small
- added D4: 5V_ST, symbol Device:LED_Small
- added F1: 2A, symbol Device:Fuse
- added F2: 5A, symbol Device:Fuse
- added FB1: FerriteBead_Small, symbol Device:FerriteBead_Small
- added J2: J_PSU_IN, symbol Connector_Generic:Conn_02x02_Counter_Clockwise
- added R1, R2: R_Shunt, symbol Device:R_Shunt
- added R10, R12, R7, R8, R9: 1K, symbol Device:R_Small
- added R11, R5: 10K, symbol Device:R_Small
- added R13: 4.7K, symbol Device:R_Small
- added R14: 1.5K, symbol Device:R_Small
- added R3: 10k, symbol Device:R_Small
- added R4: 33K, symbol Device:R_Small
- added R6: 13K, symbol Device:R_Small
- added TH1: Thermistor_NTC, symbol Device:Thermistor_NTC
- added U1, U2: INA180A2, Package_TO_SOT_SMD:SOT-23-5, symbol Amplifier_Current:INA180A2
- added U3: STM32F103C8Tx, Package_QFP:LQFP-48_7x7mm_P0.5mm, symbol MCU_ST_STM32F1:STM32F103C8Tx
Connections:
- new net: D3.2 (A), R13.1
- new net: R5.2, R6.1, R8.1
- new net: R9.2, U1.1
- new net: R1.2, U1.3 (+)
- new net: R1.3, U1.4 (-)
- new net: C8.1, C9.2, FB1.2, U3.9 (VDDA)
- new net: R3.1, R4.2, R7.1
- new net: R10.2, U2.1
- new net: R2.2, U2.3 (+)
- new net: R2.3, U2.4 (-)
- new net: R11.2, R12.1, TH1.1
- new net: D4.2 (A), R14.1
- new net +12V: D3.1 (K), R1.4, R4.1
- new net +12V_FUSED: F2.1, R1.1
- new net +12V_IN: D2.C, F2.2, J2.1 (Pin_1)
- new net +3.3V: C3.2, C5.2, FB1.1, R11.1, U1.5 (V+), U2.5 (V+)
- new net +5V: D4.1 (K), R2.4, R5.1
- new net +5V_FUSED: F1.2, R2.1
- new net +5V_IN: D1.C, F1.1, J2.4 (Pin_4)
- new net 12V_READ_ADC: C1.1, R7.2, U3.10 (PA0)
- new net 5V_READ_ADC: C2.1, R8.2, U3.11 (PA1)
- new net GND: C1.2, C2.2, C3.1, C4.2, C5.1, C6.2, C7.2, C8.2, C9.1, D1.A, D2.A, J2.2 (Pin_2), J2.3 (Pin_3), R13.2, R14.2, R3.2, R6.2, TH1.2, U1.2 (GND), U3.23 (VSS), U3.35 (VSS), U3.47 (VSS), U3.8 (VSSA)
- new net I_12V_ADC: C4.1, R9.1, U3.12 (PA2)
- new net I_5V_ADC: C6.1, R10.1, U3.13 (PA3)
- new net NTC_ADC: C7.1, R12.2, U3.16 (PA6)
Other:
- note added: "Current Sensing"
- note added: "Power Indicators"
- note added: "Power/ TVS Protection / Fusing"
- note added: "Temperature Sensing"
- note added: "Voltage Sensing"

Commit message: feat(pcb): complete PDU schematic — standard block imported, ERC clean (#202)
Import the shared STM32 CAN-node block and finish wiring:

- CAN: SN65HVD230 (Rs->GND high-speed), J_BUS_OUT (8-pin power+CAN),
  CAN-in (2x2), 120R term jumper — split-source injection
- Power reg: AMS1117-3.3 (10uF in / 22uF out)
- MCU support: 8MHz xtal, BOOT0 pulldown, NRST reset, SWD header,
  per-pin VDD decoupling, diag-serial header, mounting holes
- Status LEDs: MCU-driven PANEL_RED/GREEN + rail-present indicators
- PWR_FLAG on all externally-sourced rails + GND; 10uF rail bulk

ERC passes clean. Remaining: footprints (verify shunt terminal count)
+ DRC after layout.
Parts:
- removed D3: 12V_ST, symbol Device:LED_Small
- removed D4: 5V_ST, symbol Device:LED_Small
- removed R13: 4.7K, symbol Device:R_Small
- removed R14: 1.5K, symbol Device:R_Small
- added C10, C12, C14, C15, C16, C18: 100nF, Capacitor_SMD:C_0805_2012Metric, symbol Device:C
- added C11: 10uF, Capacitor_SMD:CP_Elec_4x5.4, symbol Device:C_Polarized
- added C13: 22uF, Capacitor_SMD:CP_Elec_4x5.4, symbol Device:C_Polarized
- added C17: 100nf, Capacitor_SMD:C_0805_2012Metric, symbol Device:C
- added C19, C20: 22pF, Capacitor_SMD:C_0805_2012Metric, symbol Device:C
- added C21, C22: 10uF, Capacitor_SMD:C_0805_2012Metric, symbol Device:C
- added D5, D7: GREEN, LED_SMD:LED_0805_2012Metric, symbol Device:LED
- added D6: RED, LED_SMD:LED_0805_2012Metric, symbol Device:LED
- added D8: 5V_ST, LED_SMD:LED_0805_2012Metric, symbol Device:LED
- added D9: 12V_ST, LED_SMD:LED_0805_2012Metric, symbol Device:LED
- added H1, H2, H3, H4: MountingHole, MountingHole:MountingHole_2.7mm_M2.5, symbol Mechanical:MountingHole
- added J1: J_DIAG, Connector_JST:JST_XH_B3B-XH-A_1x03_P2.50mm_Vertical, symbol Connector_Generic:Conn_01x03
- added J3: J_BUS_IN, symbol Connector_Generic:Conn_02x02_Counter_Clockwise
- added J5: J_CAN_TERM, Connector_PinHeader_2.54mm:PinHeader_1x02_P2.54mm_Vertical, symbol Connector_Generic:Conn_01x02
- added J7: J_SWD, Connector_PinHeader_2.54mm:PinHeader_1x05_P2.54mm_Vertical, symbol Connector_Generic:Conn_01x05
- added J9: J_BUS_OUT, Connector_Molex:Molex_Mini-Fit_Jr_5566-08A_2x04_P4.20mm_Vertical, symbol Connector_Generic:Conn_02x04_Top_Bottom
- added R13: 120, Resistor_SMD:R_0805_2012Metric, symbol Device:R
- added R14: 10k, Resistor_SMD:R_0805_2012Metric, symbol Device:R
- added R15: 1K, Resistor_SMD:R_0805_2012Metric, symbol Device:R
- added R16, R17: 3.3k, Resistor_SMD:R_0805_2012Metric, symbol Device:R
- added R18: 33, Resistor_SMD:R_0805_2012Metric, symbol Device:R
- added R19: 1.5K, Resistor_SMD:R_0805_2012Metric, symbol Device:R
- added R20: 4.7K, Resistor_SMD:R_0805_2012Metric, symbol Device:R
- added R_BOOT1: 10K, Resistor_SMD:R_0805_2012Metric, symbol Device:R
- added SW1: RESET, Button_Switch_THT:SW_PUSH_6mm, symbol Switch:SW_Push
- added U4: AMS1117-3.3, Package_TO_SOT_SMD:SOT-223-3_TabPin2, symbol Regulator_Linear:AMS1117-3.3
- added U5: SN65HVD230, Package_SO:SOIC-8_3.9x4.9mm_P1.27mm, symbol Interface_CAN_LIN:SN65HVD230
- added Y1: 8MHz, Crystal:Crystal_SMD_5032-2Pin_5.0x3.2mm, symbol Device:Crystal
- D1: footprint SMBJ5.0A:DIOM4336X265N -> OpenSkyhawk:DIOM4336X265N
- D2: footprint SMBJ12A:DIOM4336X265N -> OpenSkyhawk:DIOM4336X265N
Connections:
- net +12V: now also C22.1, D9.2 (A), J9.1 (Pin_1), J9.2 (Pin_2)
- net +3.3V: now also U3.1 (VBAT), U3.24 (VDD), U3.36 (VDD), U3.48 (VDD), C10.1, C12.1, C13.1, C14.1, C15.1, C16.1, C17.1, D5.2 (A), J7.1 (Pin_1), R14.2, U4.2 (VO), U5.3 (VCC)
- net +5V: now also C11.1, C21.1, D8.2 (A), J9.3 (Pin_3), U4.3 (VI)
- net GND: now also U2.2 (GND), C10.2, C11.2, C12.2, C13.2, C14.2, C15.2, C16.2, C17.2, C18.2, C21.2, C22.2, J1.3 (Pin_3), J3.2 (Pin_2), J3.3 (Pin_3), J7.5 (Pin_5), J9.4 (Pin_4), J9.7 (Pin_7), J9.8 (Pin_8), R15.2, R16.2, R17.2, R19.2, R20.2, R_BOOT1.2, SW1.1, U4.1 (GND), U5.2 (GND), U5.8 (Rs)
- net PANEL_RED: now reaches U3.27 (PB14)
- net PANEL_RED: now also D6.2 (A)
- net PANEL_GREEN: now reaches U3.28 (PB15)
- net PANEL_GREEN: now also D7.2 (A)
- net DIAG_TX: now reaches U3.30 (PA9)
- net DIAG_TX: now also J1.2 (Pin_2)
- net DIAG_RX: now reaches U3.31 (PA10)
- net DIAG_RX: now also J1.1 (Pin_1)
- net CAN_RX: now reaches U3.32 (PA11)
- net CAN_RX: now also U5.4 (R)
- net CAN_TX: now reaches U3.33 (PA12)
- net CAN_TX: now also U5.1 (D)
- net SWDIO: now reaches U3.34 (PA13)
- net SWDIO: now also R18.1
- net SWDCLK: now reaches U3.37 (PA14)
- net SWDCLK: now also J7.3 (Pin_3)
- net at U3.44 (BOOT0): now also R_BOOT1.1
- net OSC_IN: now reaches U3.5 (PD0)
- net OSC_IN: now also C20.1, Y1.2
- net OSC_OUT: now reaches U3.6 (PD1)
- net OSC_OUT: now also C19.2, Y1.1
- net NRST: now reaches U3.7 (NRST)
- net NRST: now also C18.1, J7.4 (Pin_4), R14.1, SW1.2
- new net: D7.1 (K), R17.1
- new net: D9.1 (K), R20.1
- new net: C19.1, C20.2
- new net: D8.1 (K), R19.1
- new net: D6.1 (K), R16.1
- new net: J7.2 (Pin_2), R18.2
- new net: J5.1 (Pin_1), R13.2
- new net: D5.1 (K), R15.1
- new net CANH: J3.1 (Pin_1), J9.5 (Pin_5), R13.1, U5.7 (CANH)
- new net CANL: J3.4 (Pin_4), J5.2 (Pin_2), J9.6 (Pin_6), U5.6 (CANL)
- no-connect marks 0 -> 23
Other:
- note added: "CAN Bus"
- note added: "CAN Bus In"
- note added: "CAN Bus Out"
- note added: "Diagnostics Serial"
- note added: "PanelGroup Status"
- note added: "Power"
- note added: "Power Regulation"
- note added: "Programming"
- note added: "Status LED Indicators"
- note removed: "Power Indicators"
- moved on the sheet: C5, C6, C7, C8, C9, FB1, R10, R11, R12, R2, TH1, U2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

Commit message: feat(pcb): PDU layout complete — routed, DRC-clean, 3D models (#202)
Full PCB layout for the per-console Power Distribution Unit:

- 2-layer, GND plane stitched top/bottom; power lanes input->output
- Shunt finalized to CSRF2512FT10L0 (2512, 2-terminal, stock
  R_2512 footprint; Kelvin via layout) — replaces the 2728 HoRCG
- Custom footprints: XFCN XF-508P-B-B MINI fuse holder + SMBJ TVS,
  with 3D models (fuse STEP + Molex Mini-Fit Jr STEPs in OS_3DModels)
- Silkscreen: connector pinouts, fuse ratings, LED/CAN labels, branding
- ERC 0/0, DRC 0/0 (verified via kicad-cli)

DESIGN-NOTES: final BOM w/ LCSC numbers, ADC map, CAN-node reuse,
firmware calibration architecture (per-board VDDA + INA zero-cal,
CAN/serial trigger, flash-page storage).

Next: enclosure (FreeCAD) + PDU firmware.
Parts:
- removed J2: J_PSU_IN, symbol Connector_Generic:Conn_02x02_Counter_Clockwise
- removed R1, R2: R_Shunt, symbol Device:R_Shunt
- added J1: J_PSU_IN, symbol Connector_Generic:Conn_02x02_Odd_Even
- added R1, R2: 10m, Resistor_SMD:R_2512_6332Metric, symbol Device:R
- C1: renamed from C3; footprint (none) -> Capacitor_SMD:C_0805_2012Metric
- C13: renamed from C17; value 100nf -> 100nF
- C19: renamed from C9; footprint (none) -> Capacitor_SMD:C_0805_2012Metric
- C2: renamed from C5; footprint (none) -> Capacitor_SMD:C_0805_2012Metric
- C20: renamed from C8; footprint (none) -> Capacitor_SMD:C_0805_2012Metric
- C3: renamed from C7; footprint (none) -> Capacitor_SMD:C_0805_2012Metric
- C4: renamed from C1; footprint (none) -> Capacitor_SMD:C_0805_2012Metric
- C5: renamed from C2; footprint (none) -> Capacitor_SMD:C_0805_2012Metric
- C6: footprint (none) -> Capacitor_SMD:C_0805_2012Metric
- C7: renamed from C4; footprint (none) -> Capacitor_SMD:C_0805_2012Metric
- F1: renamed from F2; footprint (none) -> OpenSkyhawk:FUSE-TH_4P-L16.0-W6.7
- F2: renamed from F1; footprint (none) -> OpenSkyhawk:FUSE-TH_4P-L16.0-W6.7
- FB1: footprint (none) -> Inductor_SMD:L_0805_2012Metric
- J3: footprint (none) -> Connector_Molex:Molex_Mini-Fit_Jr_5566-04A_2x02_P4.20mm_Vertical
- R10: renamed from R8; footprint (none) -> Resistor_SMD:R_0805_2012Metric
- R11: renamed from R10; footprint (none) -> Resistor_SMD:R_0805_2012Metric
- R12: renamed from R9; footprint (none) -> Resistor_SMD:R_0805_2012Metric
- R16, R17: value 3.3k -> 1K
- R3: renamed from R11; footprint (none) -> Resistor_SMD:R_0805_2012Metric
- R4, R5: footprint (none) -> Resistor_SMD:R_0805_2012Metric
- R6: renamed from R3; footprint (none) -> Resistor_SMD:R_0805_2012Metric
- R7: renamed from R6; footprint (none) -> Resistor_SMD:R_0805_2012Metric
- R8: renamed from R12; footprint (none) -> Resistor_SMD:R_0805_2012Metric
- R9: renamed from R7; footprint (none) -> Resistor_SMD:R_0805_2012Metric
- TH1: footprint (none) -> Resistor_SMD:R_1206_3216Metric
- renumbered C11 to C10, C13 to C11, C10 to C14, C18 to C15, C14 to C16, C15 to C17, C16 to C18, C19 to C21, C20 to C22, C21 to C8, C22 to C9, D2 to D1, D1 to D2, D9 to D3, D8 to D4, J9 to J2, J7 to J4, J1 to J6, R20 to R13, R19 to R14, R13 to R19, R14 to R20, U4 to U3, U5 to U4, U3 to U5
Connections:
- net +12V: now also U1.4 (-), R1.2
- net +12V_FUSED: now also U1.3 (+), R1.1
- net +12V_IN: now also J1.1 (Pin_1)
- net +5V: now also U2.4 (-), R2.2
- net +5V_FUSED: now also U2.3 (+), R2.1
- net +5V_IN: now also J1.2 (Pin_2)
- net GND: now also J1.3 (Pin_3), J1.4 (Pin_4)

Commit message: updated value for the TVS diode. (#219)
Parts:
- D2: value SMBJ5.0A -> SMBJ6.0A
Changed lines of the file:
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@@
 			)
 		)
-		(property "Value" "SMBJ5.0A"
+		(property "Value" "SMBJ6.0A"
 			(at 73.66 39.37 0)
 			(show_name no)

Commit message: feat(pcb): label LCSC/tolerance/voltage on Right_Nav + PDU schematics
Populate LCSC, Tolerance, and Rating (voltage/power) fields across the four
fabbed boards, sourced from InvenTree + the board tickets and PDU DESIGN-NOTES.
Values corrected to the selected part (100nF 50V, resistors 1%, AMS1117
C6186 -> C347222, 10uF split 25V/35V by +12V rail).

- PDU: dividers 0.1% (C2828767/C865184/C406725/C110774), J1 Mini-Fit 4-pin
  C20608114, D3/D4 green, C9 35V on +12V (SMBJ12A clamp margin).
- ARC-51A: MCP23017 C506653, TCA9548 C130026, J9 XH-8 C23067548, backlight
  J8 Mini-Fit 2-pin C20608113.
- ASN-41: AMS1117 C347222, TCA9548 C130026, 10uF per-rail split, 74HC165 x4
  C22384789, 1k ADC filter C844939, backlight J8 C20608113.
- APN-153: footprints (0805 passives + XH/Mini-Fit connectors) + MCP23017
  C506653, DRV8833 C50506, 2N7002 C8545, 2.2uF C87994 (25V X5R), 10nF C1710,
  6-pin XH J2 C23067546.

Off-board panel controls (encoders, rotary switches, OLED, pot, stepper, MEM
button) excluded as connector-coupled. Pin headers (SWD, CAN_TERM) hand-
soldered, no assembly LCSC. Harness mating ends tracked in the order BOM.
Parts:
- C1, C12, C13, C14, C15, C16, C17, C18, C2, C20, C3, C4, C5, C6, C7: LCSC (none) -> C1711; Rating (none) -> 50V; Tolerance (none) -> 10%
- C10: LCSC (none) -> C3343; Rating (none) -> 25V; Tolerance (none) -> 20%
- C11: LCSC (none) -> C72502; Rating (none) -> 16V; Tolerance (none) -> 20%
- C19: LCSC (none) -> C28323; Rating (none) -> 50V; Tolerance (none) -> 10%
- C21, C22: LCSC (none) -> C1804; Rating (none) -> 50V; Tolerance (none) -> 5%
- C8: LCSC (none) -> C669099; Rating (none) -> 25V; Tolerance (none) -> 20%
- C9: LCSC (none) -> C49010152; Rating (none) -> 35V; Tolerance (none) -> 20%
- D1: LCSC (none) -> C42368008
- D2: LCSC (none) -> C5331096
- D3, D4, D5, D7: LCSC (none) -> C19171393
- D6: LCSC (none) -> C19171391
- F1, F2: LCSC (none) -> C19727305
- FB1: LCSC (none) -> C21519
- J1: footprint (none) -> Connector_Molex:Molex_Mini-Fit_Jr_5566-04A_2x02_P4.20mm_Vertical; LCSC (none) -> C20608114
- J2: LCSC (none) -> C20608116
- J3: LCSC (none) -> C20608114
- J6: LCSC (none) -> C51940188
- R1, R2: LCSC (none) -> C346481; Rating (none) -> 2W; Tolerance (none) -> 1%
- R10, R11, R12, R15, R16, R17, R8, R9: LCSC (none) -> C110774; Rating (none) -> 1/8W; Tolerance (none) -> 0.1%
- R13: LCSC (none) -> C844941; Rating (none) -> 1/8W; Tolerance (none) -> 1%
- R14: LCSC (none) -> C49254235; Rating (none) -> 1/8W; Tolerance (none) -> 1%
- R18: LCSC (none) -> C2090807; Rating (none) -> 1/8W; Tolerance (none) -> 1%
- R19: LCSC (none) -> C844816; Rating (none) -> 1/8W; Tolerance (none) -> 1%
- R20, R6: LCSC (none) -> C406725; Rating (none) -> 1/8W; Tolerance (none) -> 0.1%
- R3, R5, R_BOOT1: LCSC (none) -> C844937; Rating (none) -> 1/8W; Tolerance (none) -> 1%
- R4: LCSC (none) -> C2828767; Rating (none) -> 1/8W; Tolerance (none) -> 0.1%
- R7: LCSC (none) -> C865184; Rating (none) -> 1/8W; Tolerance (none) -> 0.1%
- SW1: LCSC (none) -> C2939600
- TH1: LCSC (none) -> C52155460; Tolerance (none) -> 1%
- U1, U2: LCSC (none) -> C192764
- U3: LCSC (none) -> C347222
- U4: LCSC (none) -> C12084
- U5: LCSC (none) -> C8734
- Y1: LCSC (none) -> C20617997

Commit message: feat(pcb): label base boards + PDU 1k downgrade to 1%
Extends the LCSC/tolerance/voltage labeling to the two base boards and
corrects a PDU over-spec.

- Gateway_Bridge, PanelGroup_Base: LCSC + tolerance + voltage on all
  parts (footprints already present). 10uF split 25V/35V by +12V rail.
  RP2040-Zero left blank (module, ordered separately, no LCSC); pin
  headers hand-soldered (no assembly LCSC).
- PDU: R8-R12/R15-R17 (1k series/anti-alias) downgraded C110774 0.1%
  -> C844939 1%. Precision belongs only on the divider ratio resistors
  (33k/13k/10k); the series 1k sit into high-Z ADC pins where 1% reads
  identically. Drops the precision C110774 from the board entirely.
- DESIGN-NOTES: record the 1k downgrade + the order-time shunt upgrade
  (C346481 100ppm -> C500740 25ppm).
Parts:
- R10, R11, R12, R15, R16, R17, R8, R9: LCSC C110774 -> C844939; Tolerance 0.1% -> 1%
Changed lines of the file:
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@@
 			)
 		)
-		(property "Tolerance" "0.1%"
+		(property "Tolerance" "1%"
 			(at 246.38 157.48 0)
 			(hide yes)
@@
 			)
 		)
-		(property "LCSC" "C110774"
+		(property "LCSC" "C844939"
 			(at 246.38 157.48 0)
 			(hide yes)
@@
 			)
 		)
-		(property "Tolerance" "0.1%"
+		(property "Tolerance" "1%"
 			(at 57.15 96.52 0)
 			(hide yes)
@@
 			)
 		)
-		(property "LCSC" "C110774"
+		(property "LCSC" "C844939"
 			(at 57.15 96.52 0)
 			(hide yes)
@@
 			)
 		)
-		(property "Tolerance" "0.1%"
+		(property "Tolerance" "1%"
 			(at 67.31 204.47 0)
 			(hide yes)
@@
 			)
 		)
-		(property "LCSC" "C110774"
+		(property "LCSC" "C844939"
 			(at 67.31 204.47 0)
 			(hide yes)
@@
 			)
 		)
-		(property "Tolerance" "0.1%"
+		(property "Tolerance" "1%"
 			(at 53.34 255.27 0)
 			(hide yes)
@@
 			)
 		)
-		(property "LCSC" "C110774"
+		(property "LCSC" "C844939"
 			(at 53.34 255.27 0)
 			(hide yes)
@@
 			)
 		)
-		(property "Tolerance" "0.1%"
+		(property "Tolerance" "1%"
 			(at 208.28 156.21 0)
 			(hide yes)
@@
 			)
 		)
-		(property "LCSC" "C110774"
+		(property "LCSC" "C844939"
 			(at 208.28 156.21 0)
 			(hide yes)
@@
 			)
 		)
-		(property "Tolerance" "0.1%"
+		(property "Tolerance" "1%"
 			(at 57.15 73.66 0)
 			(hide yes)
@@
 			)
 		)
-		(property "LCSC" "C110774"
+		(property "LCSC" "C844939"
 			(at 57.15 73.66 0)
 			(hide yes)
@@
 			)
 		)
-		(property "Tolerance" "0.1%"
+		(property "Tolerance" "1%"
 			(at 226.06 157.48 0)
 			(hide yes)
@@
 			)
 		)
-		(property "LCSC" "C110774"
+		(property "LCSC" "C844939"
 			(at 226.06 157.48 0)
 			(hide yes)
@@
 			)
 		)
-		(property "Tolerance" "0.1%"
+		(property "Tolerance" "1%"
 			(at 71.12 156.21 0)
 			(hide yes)
@@
 			)
 		)
-		(property "LCSC" "C110774"
+		(property "LCSC" "C844939"
 			(at 71.12 156.21 0)
 			(hide yes)

Commit message: chore(pcb): normalize passive value-string case fleet-wide
Cosmetic cleanup — standardize resistor/cap value strings so identical
parts stop showing as separate BOM lines. Value = magnitude only;
tolerance + LCSC carry the precision distinction.

- 10K -> 10k, 4.7K -> 4.7k, 100K -> 100k (lowercase SI k)
- 100nf -> 100nF
- 69 symbols across all 6 boards (ASN-41, ARC-51A, APN-153, PDU,
  Gateway_Bridge, PanelGroup_Base). ERC 0/0 on all.

No functional/footprint/LCSC change. PDU generic 10k and precision
divider 10k now both read "10k", distinguished by tolerance (1% vs 0.1%).
Parts:
- R13: value 4.7K -> 4.7k
- R3, R5, R_BOOT1: value 10K -> 10k
Changed lines of the file:
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@@
 			)
 		)
-		(property "Value" "4.7K"
+		(property "Value" "4.7k"
 			(at 182.88 157.48 90)
 			(show_name no)
@@
 			)
 		)
-		(property "Value" "10K"
+		(property "Value" "10k"
 			(at 43.18 93.98 90)
 			(show_name no)
@@
 			)
 		)
-		(property "Value" "10K"
+		(property "Value" "10k"
 			(at 41.91 252.73 90)
 			(show_name no)
@@
 			)
 		)
-		(property "Value" "10K"
+		(property "Value" "10k"
 			(at 318.77 78.74 0)
 			(show_name no)

Commit message: chore(pcb): normalize remaining uppercase-K resistor values
Completes the value-string cleanup — the first pass only caught the
case-duplicate values (10K/4.7K/100K). This fixes the uppercase-K values
that had no lowercase twin: 1K, 1.5K, 13K, 33K -> lowercase k.

13 symbols. All 6 boards now fully SI-consistent (lowercase k, uppercase
F); zero remaining violations, ERC 0/0.
Parts:
- R10, R11, R12, R15, R16, R17, R8, R9: value 1K -> 1k
- R14: value 1.5K -> 1.5k
- R4: value 33K -> 33k
- R7: value 13K -> 13k
Changed lines of the file:
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@@
 			)
 		)
-		(property "Value" "1K"
+		(property "Value" "1k"
 			(at 248.92 158.75 90)
 			(show_name no)
@@
 			)
 		)
-		(property "Value" "13K"
+		(property "Value" "13k"
 			(at 50.8 104.1399 0)
 			(show_name no)
@@
 			)
 		)
-		(property "Value" "1K"
+		(property "Value" "1k"
 			(at 57.15 93.98 90)
 			(show_name no)
@@
 			)
 		)
-		(property "Value" "1K"
+		(property "Value" "1k"
 			(at 66.0401 207.01 0)
 			(show_name no)
@@
 			)
 		)
-		(property "Value" "1K"
+		(property "Value" "1k"
 			(at 53.34 252.73 90)
 			(show_name no)
@@
 			)
 		)
-		(property "Value" "1.5K"
+		(property "Value" "1.5k"
 			(at 196.85 157.48 90)
 			(show_name no)
@@
 			)
 		)
-		(property "Value" "1K"
+		(property "Value" "1k"
 			(at 210.82 157.48 90)
 			(show_name no)
@@
 			)
 		)
-		(property "Value" "1K"
+		(property "Value" "1k"
 			(at 57.15 71.12 90)
 			(show_name no)
@@
 			)
 		)
-		(property "Value" "33K"
+		(property "Value" "33k"
 			(at 43.18 71.12 90)
 			(show_name no)
@@
 			)
 		)
-		(property "Value" "1K"
+		(property "Value" "1k"
 			(at 228.6 158.75 90)
 			(show_name no)
@@
 			)
 		)
-		(property "Value" "1K"
+		(property "Value" "1k"
 			(at 69.8501 158.75 0)
 			(show_name no)
