File: PCB/Base/Power/PDU/PDU.kicad_sch (KiCad schematic)
At the start: 71 parts, among them J1 J_PSU_IN, J2 J_BUS_OUT, J3 J_BUS_IN, J4 J_SWD, J5 J_CAN_TERM, J6 J_DIAG, SW1 RESET, U1 INA180A2, U2 INA180A2, U3 AMS1117-3.3, U4 SN65HVD230, U5 STM32F103C8Tx, Y1 8MHz

Commit message: feat(pcb): label LCSC/tolerance/voltage across fleet boards (Right_Nav + PDU + base) (#235)
Populates **LCSC part number + tolerance + voltage** fields across all
six fleet boards, so each schematic drives an orderable BOM.

## Boards labeled (ERC 0/0 on all)
- **Right_Nav:** ASN-41, ARC-51A, APN-153
- **Power:** PDU
- **Base:** Gateway_Bridge, PanelGroup_Base

## What it does
- LCSC + tolerance + voltage on every assembled part, corrected to the
selected part (100nF 50V, resistors 1%, AMS1117 C6186→C347222, 10µF
split 25V/35V by +12V rail).
- Off-board panel controls (encoders, rotary switches, OLED, pot,
stepper, MEM button) left blank — connector-coupled, no assembly LCSC.
- Pin headers hand-soldered; RP2040-Zero left blank (module, sourced
separately).

## Design corrections captured here
- **PDU 1k series/anti-alias → 1%** (C110774 0.1% → C844939): precision
belongs only on the divider ratio resistors (33k/13k/10k); the series 1k
sit into high-Z ADC pins where 1% is identical. Drops the precision part
from the board.
- **DESIGN-NOTES:** records the 1k downgrade + the order-time shunt
upgrade (C346481 ±100ppm → C500740 ±25ppm, drop-in 2512).

## Not in this PR (follow-ups)
- Fleet component **standardization** (10µF-bulk→electrolytic,
consolidate to single 35V value, IPN convention) — separate pass.
- InvenTree backfill of the new SKUs.
Parts:
- C1, C12, C13, C14, C15, C16, C17, C18, C2, C20, C3, C4, C5, C6, C7: LCSC (none) -> C1711; Rating (none) -> 50V; Tolerance (none) -> 10%
- C10: LCSC (none) -> C3343; Rating (none) -> 25V; Tolerance (none) -> 20%
- C11: LCSC (none) -> C72502; Rating (none) -> 16V; Tolerance (none) -> 20%
- C19: LCSC (none) -> C28323; Rating (none) -> 50V; Tolerance (none) -> 10%
- C21, C22: LCSC (none) -> C1804; Rating (none) -> 50V; Tolerance (none) -> 5%
- C8: value 10uF -> 100nF; LCSC (none) -> C1711; Rating (none) -> 50V; Tolerance (none) -> 10%
- C9: LCSC (none) -> C49010152; Rating (none) -> 35V; Tolerance (none) -> 20%
- D1: LCSC (none) -> C42368008
- D2: Check_prices https://www.snapeda.com/parts/SMBJ5.0A/taiwan/view-part/?re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 -> (none); LCSC (none) -> C5331096; MF Taiwan Semiconductor -> MSKSEMI; MP SMBJ5.0A -> SMBJ6.0A; PARTREV F2102 -> NA; Package SMD-2 Taiwan Semiconductor -> SMD-2; Purchase-URL https://www.snapeda.com/api/url_track_click_mouser/?unipart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 -> https://www.lcsc.com/product-detail/TVS_Diodes_MSKSEMI_SMBJ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; SnapEDA_Link https://www.snapeda.com/parts/SMBJ5.0A/taiwan/view-part/?re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 -> (none)
- D3: value 12V_ST -> GREEN; LCSC (none) -> C19171393
- D4: value 5V_ST -> GREEN; LCSC (none) -> C19171393
- D5, D7: LCSC (none) -> C19171393
- D6: LCSC (none) -> C19171391
- F1, F2: LCSC (none) -> C19727305
- FB1: LCSC (none) -> C21519
- J1: footprint (none) -> Connector_Molex:Molex_Mini-Fit_Jr_5566-04A_2x02_P4.20mm_Vertical; LCSC (none) -> C20608114
- J2: LCSC (none) -> C20608116
- J3: LCSC (none) -> C20608114
- J6: LCSC (none) -> C51940188
- R1, R2: LCSC (none) -> C346481; Rating (none) -> 2W; Tolerance (none) -> 1%
- R10, R11, R12, R15, R16, R17, R8, R9: value 1K -> 1k; LCSC (none) -> C844939; Rating (none) -> 1/8W; Tolerance (none) -> 1%
- R13: value 4.7K -> 4.7k; LCSC (none) -> C844941; Rating (none) -> 1/8W; Tolerance (none) -> 1%
- R14: value 1.5K -> 1.5k; LCSC (none) -> C49254235; Rating (none) -> 1/8W; Tolerance (none) -> 1%
- R18: LCSC (none) -> C2090807; Rating (none) -> 1/8W; Tolerance (none) -> 1%
- R19: LCSC (none) -> C844816; Rating (none) -> 1/8W; Tolerance (none) -> 1%
- R20, R6: LCSC (none) -> C406725; Rating (none) -> 1/8W; Tolerance (none) -> 0.1%
- R3, R5, R_BOOT1: value 10K -> 10k; LCSC (none) -> C844937; Rating (none) -> 1/8W; Tolerance (none) -> 1%
- R4: value 33K -> 33k; LCSC (none) -> C2828767; Rating (none) -> 1/8W; Tolerance (none) -> 0.1%
- R7: value 13K -> 13k; LCSC (none) -> C865184; Rating (none) -> 1/8W; Tolerance (none) -> 0.1%
- SW1: LCSC (none) -> C2939600
- TH1: LCSC (none) -> C52155460; Tolerance (none) -> 1%
- U1, U2: LCSC (none) -> C192764
- U3: LCSC (none) -> C347222
- U4: LCSC (none) -> C12084
- U5: LCSC (none) -> C8734
- Y1: LCSC (none) -> C20617997
