File: PCB/Base/Power/PDU/PDU.kicad_sch (KiCad schematic)
At the start: 71 parts, among them J1 J_PSU_IN, J2 J_BUS_OUT, J3 J_BUS_IN, J4 J_SWD, J5 J_CAN_TERM, J6 J_DIAG, SW1 RESET, U1 INA180A2, U2 INA180A2, U3 AMS1117-3.3, U4 SN65HVD230, U5 STM32F103C8Tx, Y1 8MHz

Commit message: refactor(pcb): consolidate ceramic 10uF to single 35V part
The 10uF ceramic 0805 caps were split across two SKUs — C669099 (25V)
and C49010152 (35V) — distinguished only by rail. Standardize all 8
ceramic positions to the 35V part (C49010152); 35V covers the 25V
positions and collapses the BOM to one ceramic 10uF value.

Electrolytic 10uF (C3343) unchanged. Aluminum-bulk replacement deferred
to a future round. 8 caps across all 6 boards, ERC 0/0.
Parts:
- C8: LCSC C669099 -> C49010152; Rating 25V -> 35V
Changed lines of the file:
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@@
 			)
 		)
-		(property "Rating" "25V"
+		(property "Rating" "35V"
 			(at 111.76 40.64 0)
 			(hide yes)
@@
 			)
 		)
-		(property "LCSC" "C669099"
+		(property "LCSC" "C49010152"
 			(at 111.76 40.64 0)
 			(hide yes)

Commit message: chore(pcb): PDU status LEDs value=GREEN, function in Description
D3/D4 were labeled by function (12V_ST/5V_ST) in the Value field, which
split them from the other green LEDs in the BOM. Value now = GREEN (part
identity, groups correctly), function moved to Description ("12V/5V status
LED"). All fleet LEDs now color-named + BOM-consistent. ERC 0/0.
Parts:
- D3: value 12V_ST -> GREEN
- D4: value 5V_ST -> GREEN
Changed lines of the file:
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@@
 			)
 		)
-		(property "Value" "12V_ST"
+		(property "Value" "GREEN"
 			(at 177.8 144.78 0)
 			(show_name no)
@@
 			)
 		)
-		(property "Description" "Light emitting diode"
+		(property "Description" "12V status LED"
 			(at 180.34 147.32 0)
 			(hide yes)
@@
 			)
 		)
-		(property "Value" "5V_ST"
+		(property "Value" "GREEN"
 			(at 191.77 144.78 0)
 			(show_name no)
@@
 			)
 		)
-		(property "Description" "Light emitting diode"
+		(property "Description" "5V status LED"
 			(at 194.31 147.32 0)
 			(hide yes)

Commit message: fix(pcb): correct SMBJ6.0A TVS metadata on PDU/base boards
D2 (PDU), D6 (Gateway_Bridge), D3 (PanelGroup_Base) carried stale
SnapEDA metadata from the original SMBJ5.0A (Taiwan Semiconductor)
symbol after the value was swapped to the 6.0A part. Value + LCSC
(C5331096) were already correct; this aligns the rest so BOM/inventory
exports agree with InvenTree:
- MF Taiwan Semiconductor -> MSKSEMI (actual mfr of C5331096)
- MP SMBJ5.0A -> SMBJ6.0A (PDU; already correct on base boards)
- Description 5V -> 6V
- Purchase-URL -> LCSC product page; clear stale SnapEDA links,
  Taiwan-Semi PARTREV/Package refs

ERC clean on all three.
Parts:
- D2: Check_prices https://www.snapeda.com/parts/SMBJ5.0A/taiwan/view-part/?re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 -> (none); MF Taiwan Semiconductor -> MSKSEMI; MP SMBJ5.0A -> SMBJ6.0A; PARTREV F2102 -> NA; Package SMD-2 Taiwan Semiconductor -> SMD-2; Purchase-URL https://www.snapeda.com/api/url_track_click_mouser/?unipart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 -> https://www.lcsc.com/product-detail/TVS_Diodes_MSKSEMI_SMBJ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; SnapEDA_Link https://www.snapeda.com/parts/SMBJ5.0A/taiwan/view-part/?re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 -> (none)
Changed lines of the file:
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@@
 			)
 		)
-		(property "Description" "600W, 5V, Unidirectional, TVS"
+		(property "Description" "600W, 6V, Unidirectional, TVS"
 			(at 76.2 41.91 0)
 			(hide yes)
@@
 			)
 		)
-		(property "MF" "Taiwan Semiconductor"
+		(property "MF" "MSKSEMI"
 			(at 76.2 41.91 0)
 			(hide yes)
@@
 			)
 		)
-		(property "Package" "SMD-2 Taiwan Semiconductor"
+		(property "Package" "SMD-2"
 			(at 76.2 41.91 0)
 			(hide yes)
@@
 			)
 		)
-		(property "Check_prices" "https://www.snapeda.com/parts/SMBJ5.0A/taiwan/view-part/?ref=eda"
+		(property "Check_prices" ""
 			(at 76.2 41.91 0)
 			(hide yes)
@@
 			)
 		)
-		(property "PARTREV" "F2102"
+		(property "PARTREV" "NA"
 			(at 76.2 41.91 0)
 			(hide yes)
@@
 			)
 		)
-		(property "SnapEDA_Link" "https://www.snapeda.com/parts/SMBJ5.0A/taiwan/view-part/?ref=snap"
+		(property "SnapEDA_Link" ""
 			(at 76.2 41.91 0)
 			(hide yes)
@@
 			)
 		)
-		(property "MP" "SMBJ5.0A"
+		(property "MP" "SMBJ6.0A"
 			(at 76.2 41.91 0)
 			(hide yes)
@@
 			)
 		)
-		(property "Purchase-URL" "https://www.snapeda.com/api/url_track_click_mouser/?unipart_id=1860032&manufacturer=Taiwan Semiconductor&part_name=SMBJ5.0A&search_term=smbj5.0a"
+		(property "Purchase-URL" "https://www.lcsc.com/product-detail/TVS_Diodes_MSKSEMI_SMBJ6.0A_C5331096.html"
 			(at 76.2 41.91 0)
 			(hide yes)

Commit message: fix(pcb): re-value AMS1117 input ceramic 10uF->100nF (ASN/PDU/Gate/Pane)
The AMS1117 +5V input carried two bulk caps (10uF ceramic + 10uF elec)
and no HF bypass. Re-value the redundant 10uF ceramic to 100nF (reuse
C1711, 0805 unchanged) so each input = 10uF elec bulk + 100nF ceramic
HF = standard LDO input. No footprint/symbol change; ERC clean.
Frees another 10uF/35V ceramic and closes the missing-input-HF gap.
Parts:
- C8: value 10uF -> 100nF; LCSC C49010152 -> C1711; Rating 35V -> 50V; Tolerance 20% -> 10%
Changed lines of the file:
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@@
 			)
 		)
-		(property "Value" "10uF"
+		(property "Value" "100nF"
 			(at 115.57 41.9099 0)
 			(show_name no)
@@
 			)
 		)
-		(property "Rating" "35V"
+		(property "Rating" "50V"
 			(at 111.76 40.64 0)
 			(hide yes)
@@
 			)
 		)
-		(property "Tolerance" "20%"
+		(property "Tolerance" "10%"
 			(at 111.76 40.64 0)
 			(hide yes)
@@
 			)
 		)
-		(property "LCSC" "C49010152"
+		(property "LCSC" "C1711"
 			(at 111.76 40.64 0)
 			(hide yes)

Commit message: feat(pcb): add descriptive IPN field to all on-board symbols (#238 Phase 3) (#239)
Phase 3 of the IPN convention (#238): adds a stable, descriptive
**Internal Part Number** to every on-board symbol, co-equal with LCSC.
BOMs now anchor on a fixed identity; the LCSC can change with
availability without altering the part's identity.

## What changed
- **352 symbols** across all 6 boards (multi-sheet aware) get an `IPN`
field. **51 distinct IPNs.** ERC clean fleet-wide.
- **Off-board controls** (encoders/switches/pots/OLED/stepper — no
footprint, connector-coupled) get **no IPN**, per the standing off-board
exclusion. On-board modules (RP2040-ZERO) and the RESET tact switch
**do** get IPNs.
- `.gitignore`: FreeCAD backups (`*.FCBak`/`*.FCStd1`) + KiCad ERC/DRC
reports (`*-erc.rpt`/`*-drc.rpt`).

## Scheme (descriptive, locked in #238)
`RES-10K-1PCT-0805` · `CAP-CER-100NF-50V-0805` · `CAP-ELEC-22UF-16V-D4`
· `IC-STM32F103C8-LQFP` · `CONN-XH-8P` · `TVS-SMBJ12A-SMB` ·
`FUSE-HOLDER-BLADE-DIP4` · `SW-TACT-6MM` · `MOD-RP2040-ZERO`.

Resolved the 3 open encoding items: ferrite → `FB-600R-0805` (TDK
600Ω@100MHz), NTC → `NTC-10K-1206` (APV 10K), fuse holder (C19727305 is
a *holder*, not a fuse) → one `FUSE-HOLDER-BLADE-DIP4`.

## Not in this PR (later phases of #238)
- **Phase 2 — InvenTree:** set the IPN field + link SupplierParts incl
backorder alternates (one IPN → many LCSC). This is what actually
delivers the churn-proofing; needs reviewed InvenTree writes.
- **Phase 4 — order flow:** resolve IPN → in-stock LCSC at order time.

Refs #238.
Parts:
- C1, C12, C13, C14, C15, C16, C17, C18, C2, C20, C3, C4, C5, C6, C7, C8: IPN (none) -> CAP-CER-100NF-50V-0805
- C10: IPN (none) -> CAP-ELEC-10UF-25V-D4
- C11: IPN (none) -> CAP-ELEC-22UF-16V-D4
- C19: IPN (none) -> CAP-CER-1UF-50V-0805
- C21, C22: IPN (none) -> CAP-C0G-22PF-50V-0805
- C9: IPN (none) -> CAP-CER-10UF-35V-0805
- D1: IPN (none) -> TVS-SMBJ12A-SMB
- D2: IPN (none) -> TVS-SMBJ6V0A-SMB
- D3, D4, D5, D7: IPN (none) -> LED-GREEN-0805
- D6: IPN (none) -> LED-RED-0805
- F1, F2: IPN (none) -> FUSE-HOLDER-BLADE-DIP4
- FB1: IPN (none) -> FB-600R-0805
- J1, J3: IPN (none) -> CONN-MF-4P
- J2: IPN (none) -> CONN-MF-8P
- J4: IPN (none) -> CONN-HDR-5P
- J5: IPN (none) -> CONN-HDR-2P
- J6: IPN (none) -> CONN-XH-3P
- R1, R2: IPN (none) -> RES-0R010-1PCT-2512
- R10, R11, R12, R15, R16, R17, R8, R9: IPN (none) -> RES-1K-1PCT-0805
- R13: IPN (none) -> RES-4K7-1PCT-0805
- R14: IPN (none) -> RES-1K5-1PCT-0805
- R18: IPN (none) -> RES-33R-1PCT-0805
- R19: IPN (none) -> RES-120R-1PCT-0805
- R20, R6: IPN (none) -> RES-10K-0P1PCT-0805
- R3, R5, R_BOOT1: IPN (none) -> RES-10K-1PCT-0805
- R4: IPN (none) -> RES-33K-0P1PCT-0805
- R7: IPN (none) -> RES-13K-0P1PCT-0805
- SW1: IPN (none) -> SW-TACT-6MM
- TH1: IPN (none) -> NTC-10K-1206
- U1, U2: IPN (none) -> IC-INA180A2-SOT23
- U3: IPN (none) -> IC-AMS1117-3V3-SOT223
- U4: IPN (none) -> IC-SN65HVD230-SOIC
- U5: IPN (none) -> IC-STM32F103C8-LQFP
- Y1: IPN (none) -> XTAL-8MHZ-SMD5032

Commit message: feat(pcb): +12V bulk cap → 22µF/35V electrolytic reroute (#236) (#243)
## What
Replaces the **+12V bulk cap** across ASN-41, PDU, Gateway_Bridge and
PanelGroup_Base:
**10µF/35V ceramic (0805) → 22µF/35V aluminium electrolytic**
`C48971029` (`Capacitor_SMD:CP_Elec_5x5.4`).

## Why (#236)
- 10µF/35V *ceramic* on a 12V rail DC-bias-derates to ~4–6µF;
electrolytic holds full value at ~1/5 the cost.
- Footprint grows 0805 → Ø5 (35V elec), so fabbed boards get a reroute;
value taken to 22µF (same Ø5 can) for margin.

## Changes
- Symbol fields updated: IPN `CAP-ELEC-22UF-35V-D5`, LCSC `C48971029`,
Rating `35V`, Tolerance `20%`.
- **PDU (C9), Gateway_Bridge (C15), PanelGroup_Base (C15)** — rerouted
for the Ø5 land; board revision **0.1.0 → 0.2.0**.
- **ASN-41 (C15)** — unrouted, schematic only; revision **0.1.0**.

## Verification
- ERC clean (0/0) on all four boards.
- CI (KiCad PR Reports) runs ERC/DRC.

Closes #236 — the +12V ceramic→electrolytic reroute was the
consolidation's last open action; the rest is decided and applied (per
#235 + this PR).
Parts:
- removed C9: 10uF, Capacitor_SMD:C_0805_2012Metric, symbol Device:C
- added C9: 22uF, Capacitor_SMD:CP_Elec_5x5.4, symbol Device:C_Polarized_Small
Connections:
- net +12V: now also C9.1
- net GND: now also C9.2

Commit message: feat(pcb): base boards Rev 2 — PanelGroup ShiftBus remap + Gateway/PDU fab prep (#209) (#302)
Takes PanelGroup base to Rev 2 for the 74HC ShiftBus pin standard, and
prepares
Gateway_Bridge and PDU for the same fab run. Boards are ordered — JLC
`W2026093021050394`, LCSC `WM2610010130` — so this is the as-fabricated
state.

## PanelGroup base Rev 2 (#209)

- **`J_SR` ShiftBus connector** (XH-7): `SCK · MOSI · MISO · GND · 3.3V
· LOAD · LTCH`,
  with 33 Ω series termination at the driver on SCK / LOAD / LATCH.
- **Nine-pin re-map.** I²C2 interrupts move PB8/PB9 → PA8/PA15 to free
the ShiftBus
strobes; J11 positions 7 and 11 become PB2 and PC14. PB2/PC14 are chosen
so the
breakout never collides with the I²C interrupt EXTI lines, which are
shared by pin
  number across ports.
- Docs rewritten from the final netlist: `docs/_source/base-boards.md`,
plus the
  INT-pin guidance and the now-adopted `J_SR` standard.

All four Rev 1 pre-order bench checks passed, so no finding forced a Rev
2 change —
CAN at 502 kbps with ACK from a second node, I²C pull-ups and both buses
end to end,
backlight PWM at 1.000 kHz with the gate pull-downs holding through
reset. Results are
recorded in #209.

## Gateway_Bridge and PDU — fab prep

Both boards had diverged from their fabbed revision (#243 moved the +12
V bulk cap to a
22 µF/35 V electrolytic, and Gateway gained the input-rail TVS with **no
pads on the old
board**), and neither had been assembled — so both were re-fabbed rather
than built as-is.

The silkscreen gate caught three real defects on Gateway before fab:

- revision text still read `0.1.0`
- **J8/J9 (`J_BUS_IN`/`J_BUS_OUT`) had no pin labels at all** — 12 V and
CAN on two
  identical unkeyed Mini-Fit connectors side by side
- **J1 (`J_DIAG`, the serial console) was labelled `SDA`/`SCL`** instead
of `RX`/`TX`

Also fixed a `CAN TERM` legend implemented by overriding the footprint
`Value` field,
which raised a parity error and would have been silently erased by the
next schema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
Parts:
- R1, R2: LCSC C346481 -> C2903468; Rating 2W -> 3W
Changed lines of the file:
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@@
 			)
 		)
-		(property "Rating" "2W"
+		(property "Rating" "3W"
 			(at 34.29 156.21 0)
 			(hide yes)
@@
 			)
 		)
-		(property "LCSC" "C346481"
+		(property "LCSC" "C2903468"
 			(at 34.29 156.21 0)
 			(hide yes)
@@
 			)
 		)
-		(property "Rating" "2W"
+		(property "Rating" "3W"
 			(at 35.56 204.47 0)
 			(hide yes)
@@
 			)
 		)
-		(property "LCSC" "C346481"
+		(property "LCSC" "C2903468"
 			(at 35.56 204.47 0)
 			(hide yes)
