File: PCB/Base/Power/PDU/PDU.kicad_pcb (KiCad board)
At the start: 2 copper layers, 96.6 x 63.9 mm, 72 parts, among them J1 J_PSU_IN, J2 J_BUS_OUT, J3 J_BUS_IN, J4 J_SWD, J5 J_CAN_TERM, J6 J_DIAG, SW1 RESET, U1 INA180A2, U2 INA180A2, U3 AMS1117-3.3, U4 SN65HVD230, U5 STM32F103C8Tx, Y1 8MHz

Commit message: feat(pcb): +12V bulk cap → 22µF/35V electrolytic reroute (#236) (#243)
## What
Replaces the **+12V bulk cap** across ASN-41, PDU, Gateway_Bridge and
PanelGroup_Base:
**10µF/35V ceramic (0805) → 22µF/35V aluminium electrolytic**
`C48971029` (`Capacitor_SMD:CP_Elec_5x5.4`).

## Why (#236)
- 10µF/35V *ceramic* on a 12V rail DC-bias-derates to ~4–6µF;
electrolytic holds full value at ~1/5 the cost.
- Footprint grows 0805 → Ø5 (35V elec), so fabbed boards get a reroute;
value taken to 22µF (same Ø5 can) for margin.

## Changes
- Symbol fields updated: IPN `CAP-ELEC-22UF-35V-D5`, LCSC `C48971029`,
Rating `35V`, Tolerance `20%`.
- **PDU (C9), Gateway_Bridge (C15), PanelGroup_Base (C15)** — rerouted
for the Ø5 land; board revision **0.1.0 → 0.2.0**.
- **ASN-41 (C15)** — unrouted, schematic only; revision **0.1.0**.

## Verification
- ERC clean (0/0) on all four boards.
- CI (KiCad PR Reports) runs ERC/DRC.

Closes #236 — the +12V ceramic→electrolytic reroute was the
consolidation's last open action; the rest is decided and applied (per
#235 + this PR).
Parts:
- C8: value 10uF -> 100nF
- C9: value 10uF -> 22uF; footprint Capacitor_SMD:C_0805_2012Metric -> Capacitor_SMD:CP_Elec_5x5.4
- D2: value SMBJ5.0A -> SMBJ6.0A
- D3: value 12V_ST -> GREEN
- D4: value 5V_ST -> GREEN
- R10, R11, R12, R15, R16, R17, R8, R9: value 1K -> 1k
- R13: value 4.7K -> 4.7k
- R14: value 1.5K -> 1.5k
- R3, R5, R_BOOT1: value 10K -> 10k
- R4: value 33K -> 33k
- R7: value 13K -> 13k
- moved R9 32.2 mm to (162.8, 64.6), turned to -90 degrees
- moved R6 29.2 mm to (162.8, 61.0), turned to 90 degrees
- moved R7 28.7 mm to (166.1, 64.6), turned to -90 degrees
- moved R10 26.5 mm to (168.3, 64.6), turned to -90 degrees
- moved R4 25.3 mm to (166.1, 61.0), turned to -90 degrees
- moved R5 22.8 mm to (168.3, 60.9), turned to -90 degrees
- moved C9 19.6 mm to (173.7, 36.0), turned to 90 degrees
- moved J2 18.7 mm to (166.1, 42.5)
- moved G*** 8.09 mm to (195.3, 62.1)
Routing:
- net +12V: track 109.1 -> 68.3 mm, vias 1 -> 0
- net /5V_READ_ADC: track 77.9 -> 52.2 mm
- net /12V_READ_ADC: track 95.8 -> 70.3 mm
- net /CANH: track 78.3 -> 101.9 mm
- net +5V: track 92.1 -> 86.5 mm, vias 8 -> 9
- net GND: track 34.2 -> 30.6 mm, vias 74 -> 72
- net /CANL: track 104.9 -> 107.1 mm
Other:
- board text added: "POWER DISTRIBUTION UNIT | REVISION 0.2.0"
- board text removed: "POWER DISTRIBUTION UNIT | REVISION 0.1.0"

Commit message: fix(pcb): PDU silkscreen — revision text format and field sync (#209)
Prepares the board for the Rev 2 fab order. Silkscreen and field sync only;
no copper, footprint or netlist changes.

- Revision text reordered to "REVISION 0.2.0 | POWER DISTRIBUTION UNIT",
  matching the fleet format.
- Update PCB from Schematic, picking up the IPN field on C9.

Connector pin labels were already complete (24 pins checked against their
nets). ERC 0, DRC 0 violations, 0 unconnected, 0 schematic parity.
Other:
- board text added: "REVISION 0.2.0 | POWER DISTRIBUTION UNIT"
- board text removed: "POWER DISTRIBUTION UNIT | REVISION 0.2.0"
Changed lines of the file:
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@@
 			)
 		)
+		(property "IPN" "CAP-ELEC-22UF-35V-D5"
+			(at 0 0 90)
+			(unlocked yes)
+			(layer "F.Fab")
+			(hide yes)
+			(effects
+				(font
+					(size 1 1)
+					(thickness 0.15)
+				)
+			)
+		)
+		(property "Rating" "35V"
+			(at 0 0 90)
+			(unlocked yes)
+			(layer "F.Fab")
+			(hide yes)
+			(effects
+				(font
+					(size 1 1)
+					(thickness 0.15)
+				)
+			)
+		)
+		(property "Tolerance" "20%"
+			(at 0 0 90)
+			(unlocked yes)
+			(layer "F.Fab")
+			(hide yes)
+			(effects
+				(font
+					(size 1 1)
+					(thickness 0.15)
+				)
+			)
+		)
+		(property "LCSC" "C48971029"
+			(at 0 0 90)
+			(unlocked yes)
+			(layer "F.Fab")
+			(hide yes)
+			(effects
+				(font
+					(size 1 1)
+					(thickness 0.15)
+				)
+			)
+		)
 		(property ki_fp_filters "CP_*")
 		(sheetname "/")
@@
 		)
 	)
-	(gr_text "POWER DISTRIBUTION UNIT | REVISION 0.2.0"
-		(at 197.89 86.55 0)
+	(gr_text "REVISION 0.2.0 | POWER DISTRIBUTION UNIT"
+		(at 195.08 86.55 0)
 		(layer "B.SilkS")
 		(effects
