File: PCB/Base/Power/PDU/PDU.kicad_pcb (KiCad board)
At the start: 2 copper layers, 96.6 x 63.9 mm, 72 parts, among them J1 J_PSU_IN, J2 J_BUS_OUT, J3 J_BUS_IN, J4 J_SWD, J5 J_CAN_TERM, J6 J_DIAG, SW1 RESET, U1 INA180A2, U2 INA180A2, U3 AMS1117-3.3, U4 SN65HVD230, U5 STM32F103C8Tx, Y1 8MHz

Commit message: feat(pcb): base boards Rev 2 — PanelGroup ShiftBus remap + Gateway/PDU fab prep (#209) (#302)
Takes PanelGroup base to Rev 2 for the 74HC ShiftBus pin standard, and
prepares
Gateway_Bridge and PDU for the same fab run. Boards are ordered — JLC
`W2026093021050394`, LCSC `WM2610010130` — so this is the as-fabricated
state.

## PanelGroup base Rev 2 (#209)

- **`J_SR` ShiftBus connector** (XH-7): `SCK · MOSI · MISO · GND · 3.3V
· LOAD · LTCH`,
  with 33 Ω series termination at the driver on SCK / LOAD / LATCH.
- **Nine-pin re-map.** I²C2 interrupts move PB8/PB9 → PA8/PA15 to free
the ShiftBus
strobes; J11 positions 7 and 11 become PB2 and PC14. PB2/PC14 are chosen
so the
breakout never collides with the I²C interrupt EXTI lines, which are
shared by pin
  number across ports.
- Docs rewritten from the final netlist: `docs/_source/base-boards.md`,
plus the
  INT-pin guidance and the now-adopted `J_SR` standard.

All four Rev 1 pre-order bench checks passed, so no finding forced a Rev
2 change —
CAN at 502 kbps with ACK from a second node, I²C pull-ups and both buses
end to end,
backlight PWM at 1.000 kHz with the gate pull-downs holding through
reset. Results are
recorded in #209.

## Gateway_Bridge and PDU — fab prep

Both boards had diverged from their fabbed revision (#243 moved the +12
V bulk cap to a
22 µF/35 V electrolytic, and Gateway gained the input-rail TVS with **no
pads on the old
board**), and neither had been assembled — so both were re-fabbed rather
than built as-is.

The silkscreen gate caught three real defects on Gateway before fab:

- revision text still read `0.1.0`
- **J8/J9 (`J_BUS_IN`/`J_BUS_OUT`) had no pin labels at all** — 12 V and
CAN on two
  identical unkeyed Mini-Fit connectors side by side
- **J1 (`J_DIAG`, the serial console) was labelled `SDA`/`SCL`** instead
of `RX`/`TX`

Also fixed a `CAN TERM` legend implemented by overriding the footprint
`Value` field,
which raised a parity error and would have been silently erased by the
next schema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
Other:
- board text added: "REVISION 0.2.0 | POWER DISTRIBUTION UNIT"
- board text removed: "POWER DISTRIBUTION UNIT | REVISION 0.2.0"
Changed lines of the file:
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@@
 			)
 		)
-		(property "Rating" "2W"
+		(property "Rating" "3W"
 			(at 0 0 180)
 			(unlocked yes)
@@
 			)
 		)
-		(property "LCSC" "C346481"
+		(property "LCSC" "C2903468"
 			(at 0 0 180)
 			(unlocked yes)
@@
 			)
 		)
-		(property "Rating" "2W"
+		(property "Rating" "3W"
 			(at 0 0 180)
 			(unlocked yes)
@@
 			)
 		)
-		(property "LCSC" "C346481"
+		(property "LCSC" "C2903468"
 			(at 0 0 180)
 			(unlocked yes)
@@
 			)
 		)
+		(property "IPN" "CAP-ELEC-22UF-35V-D5"
+			(at 0 0 90)
+			(unlocked yes)
+			(layer "F.Fab")
+			(hide yes)
+			(effects
+				(font
+					(size 1 1)
+					(thickness 0.15)
+				)
+			)
+		)
+		(property "Rating" "35V"
+			(at 0 0 90)
+			(unlocked yes)
+			(layer "F.Fab")
+			(hide yes)
+			(effects
+				(font
+					(size 1 1)
+					(thickness 0.15)
+				)
+			)
+		)
+		(property "Tolerance" "20%"
+			(at 0 0 90)
+			(unlocked yes)
+			(layer "F.Fab")
+			(hide yes)
+			(effects
+				(font
+					(size 1 1)
+					(thickness 0.15)
+				)
+			)
+		)
+		(property "LCSC" "C48971029"
+			(at 0 0 90)
+			(unlocked yes)
+			(layer "F.Fab")
+			(hide yes)
+			(effects
+				(font
+					(size 1 1)
+					(thickness 0.15)
+				)
+			)
+		)
 		(property ki_fp_filters "CP_*")
 		(sheetname "/")
@@
 		)
 	)
-	(gr_text "POWER DISTRIBUTION UNIT | REVISION 0.2.0"
-		(at 197.89 86.55 0)
+	(gr_text "REVISION 0.2.0 | POWER DISTRIBUTION UNIT"
+		(at 195.08 86.55 0)
 		(layer "B.SilkS")
 		(effects
