File: PCB/Right_Console/Right_Navigation/ARC-51A_UHF/OLEDs.kicad_sch (KiCad schematic)
At the start: 10 parts, among them U4 TCA9548APWR, U5 FREQ_LOW_OLED, U6 UHF_PRE_OLED, U7 FREQ_HI_OLED

Commit message: feat(pcb): label LCSC/tolerance/voltage across fleet boards (Right_Nav + PDU + base) (#235)
Populates **LCSC part number + tolerance + voltage** fields across all
six fleet boards, so each schematic drives an orderable BOM.

## Boards labeled (ERC 0/0 on all)
- **Right_Nav:** ASN-41, ARC-51A, APN-153
- **Power:** PDU
- **Base:** Gateway_Bridge, PanelGroup_Base

## What it does
- LCSC + tolerance + voltage on every assembled part, corrected to the
selected part (100nF 50V, resistors 1%, AMS1117 C6186→C347222, 10µF
split 25V/35V by +12V rail).
- Off-board panel controls (encoders, rotary switches, OLED, pot,
stepper, MEM button) left blank — connector-coupled, no assembly LCSC.
- Pin headers hand-soldered; RP2040-Zero left blank (module, sourced
separately).

## Design corrections captured here
- **PDU 1k series/anti-alias → 1%** (C110774 0.1% → C844939): precision
belongs only on the divider ratio resistors (33k/13k/10k); the series 1k
sit into high-Z ADC pins where 1% is identical. Drops the precision part
from the board.
- **DESIGN-NOTES:** records the 1k downgrade + the order-time shunt
upgrade (C346481 ±100ppm → C500740 ±25ppm, drop-in 2512).

## Not in this PR (follow-ups)
- Fleet component **standardization** (10µF-bulk→electrolytic,
consolidate to single 35V value, IPN convention) — separate pass.
- InvenTree backfill of the new SKUs.
Parts:
- C16, C17, C18, C19: LCSC (none) -> C1711
- C20: value 10uF -> 1uF; LCSC (none) -> C28323; Rating 25V -> 50V; Tolerance 20% -> 10%
- R15: value 10K -> 10k; LCSC (none) -> C844937
Changed lines of the file:
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@@
 			)
 		)
-		(property "LCSC" ""
+		(property "LCSC" "C1711"
 			(at 15.24 2.54 0)
 			(hide yes)
@@
 			)
 		)
-		(property "Value" "10uF"
+		(property "Value" "1uF"
 			(at 85.1297 50.3073 0)
 			(show_name no)
@@
 			)
 		)
-		(property "LCSC" ""
+		(property "LCSC" "C28323"
 			(at 17.78 8.89 0)
 			(hide yes)
@@
 			)
 		)
-		(property "Tolerance" "20%"
+		(property "Tolerance" "10%"
 			(at 17.78 8.89 0)
 			(hide yes)
@@
 			)
 		)
-		(property "Rating" "25V"
+		(property "Rating" "50V"
 			(at 17.78 8.89 0)
 			(hide yes)
@@
 			)
 		)
-		(property "LCSC" ""
+		(property "LCSC" "C1711"
 			(at 16.51 50.8 0)
 			(hide yes)
@@
 			)
 		)
-		(property "LCSC" ""
+		(property "LCSC" "C1711"
 			(at 16.51 -54.61 0)
 			(hide yes)
@@
 			)
 		)
-		(property "Value" "10K"
+		(property "Value" "10k"
 			(at 53.34 81.28 90)
 			(show_name no)
@@
 			)
 		)
-		(property "LCSC" ""
+		(property "LCSC" "C844937"
 			(at 17.78 22.86 0)
 			(hide yes)
@@
 			)
 		)
-		(property "LCSC" ""
+		(property "LCSC" "C1711"
 			(at 7.62 8.89 0)
 			(hide yes)
