File: PCB/Right_Console/Right_Navigation/ARC-51A_UHF/Switches.kicad_sch (KiCad schematic)
At the start: 28 parts, among them SW1 ENC_10MHZ, SW10 ARC51_MODE, SW2 ENC_1MHZ, SW3 ENC_50KHZ, SW4 ENC_PRE, SW5 UHF_SW, SW6 SQ_DISABLE, U1 MCP23017x-x-SS

Commit message: feat(pcb): label LCSC/tolerance/voltage on Right_Nav + PDU schematics
Populate LCSC, Tolerance, and Rating (voltage/power) fields across the four
fabbed boards, sourced from InvenTree + the board tickets and PDU DESIGN-NOTES.
Values corrected to the selected part (100nF 50V, resistors 1%, AMS1117
C6186 -> C347222, 10uF split 25V/35V by +12V rail).

- PDU: dividers 0.1% (C2828767/C865184/C406725/C110774), J1 Mini-Fit 4-pin
  C20608114, D3/D4 green, C9 35V on +12V (SMBJ12A clamp margin).
- ARC-51A: MCP23017 C506653, TCA9548 C130026, J9 XH-8 C23067548, backlight
  J8 Mini-Fit 2-pin C20608113.
- ASN-41: AMS1117 C347222, TCA9548 C130026, 10uF per-rail split, 74HC165 x4
  C22384789, 1k ADC filter C844939, backlight J8 C20608113.
- APN-153: footprints (0805 passives + XH/Mini-Fit connectors) + MCP23017
  C506653, DRV8833 C50506, 2N7002 C8545, 2.2uF C87994 (25V X5R), 10nF C1710,
  6-pin XH J2 C23067546.

Off-board panel controls (encoders, rotary switches, OLED, pot, stepper, MEM
button) excluded as connector-coupled. Pin headers (SWD, CAN_TERM) hand-
soldered, no assembly LCSC. Harness mating ends tracked in the order BOM.
Parts:
- C1: LCSC (none) -> C1711
- C2: LCSC (none) -> C669099
- R22, R23, R24, R25, R26, R27, R28, R29, R30, R31, R32, R33, R42, R43, R44, R5: LCSC (none) -> C844937
- R3: LCSC (none) -> C844936
- U1: LCSC (none) -> C506653
Changed lines of the file:
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@@
 			)
 		)
-		(property "LCSC" ""
+		(property "LCSC" "C844937"
 			(at 167.64 2.54 0)
 			(hide yes)
@@
 			)
 		)
-		(property "LCSC" ""
+		(property "LCSC" "C844937"
 			(at 83.82 -64.77 0)
 			(hide yes)
@@
 			)
 		)
-		(property "LCSC" ""
+		(property "LCSC" "C669099"
 			(at 0 0 0)
 			(hide yes)
@@
 			)
 		)
-		(property "LCSC" ""
+		(property "LCSC" "C844937"
 			(at 83.82 -64.77 0)
 			(hide yes)
@@
 			)
 		)
-		(property "LCSC" ""
+		(property "LCSC" "C844937"
 			(at 215.9 1.27 0)
 			(hide yes)
@@
 			)
 		)
-		(property "LCSC" ""
+		(property "LCSC" "C844937"
 			(at 127 110.49 0)
 			(hide yes)
@@
 			)
 		)
-		(property "LCSC" ""
+		(property "LCSC" "C844937"
 			(at 120.65 46.99 0)
 			(hide yes)
@@
 			)
 		)
-		(property "LCSC" ""
+		(property "LCSC" "C1711"
 			(at 0 0 0)
 			(hide yes)
@@
 			)
 		)
-		(property "LCSC" ""
+		(property "LCSC" "C844936"
 			(at 0 0 0)
 			(hide yes)
@@
 			)
 		)
-		(property "LCSC" ""
+		(property "LCSC" "C844937"
 			(at 167.64 2.54 0)
 			(hide yes)
@@
 			)
 		)
-		(property "LCSC" ""
+		(property "LCSC" "C844937"
 			(at 0 0 0)
 			(hide yes)
@@
 			)
 		)
-		(property "LCSC" ""
+		(property "LCSC" "C844937"
 			(at 127 120.65 0)
 			(hide yes)
@@
 			)
 		)
-		(property "LCSC" ""
+		(property "LCSC" "C844937"
 			(at 120.65 2.54 0)
 			(hide yes)
@@
 			)
 		)
-		(property "LCSC" ""
+		(property "LCSC" "C506653"
 			(at 0 0 0)
 			(hide yes)
@@
 			)
 		)
-		(property "LCSC" ""
+		(property "LCSC" "C844937"
 			(at 83.82 -64.77 0)
 			(hide yes)
@@
 			)
 		)
-		(property "LCSC" ""
+		(property "LCSC" "C844937"
 			(at 120.65 2.54 0)
 			(hide yes)
@@
 			)
 		)
-		(property "LCSC" ""
+		(property "LCSC" "C844937"
 			(at 120.65 46.99 0)
 			(hide yes)
@@
 			)
 		)
-		(property "LCSC" ""
+		(property "LCSC" "C844937"
 			(at 127 115.57 0)
 			(hide yes)
@@
 			)
 		)
-		(property "LCSC" ""
+		(property "LCSC" "C844937"
 			(at 152.4 182.88 0)
 			(hide yes)
@@
 			)
 		)
-		(property "LCSC" ""
+		(property "LCSC" "C844937"
 			(at 215.9 1.27 0)
 			(hide yes)

Commit message: chore(pcb): normalize passive value-string case fleet-wide
Cosmetic cleanup — standardize resistor/cap value strings so identical
parts stop showing as separate BOM lines. Value = magnitude only;
tolerance + LCSC carry the precision distinction.

- 10K -> 10k, 4.7K -> 4.7k, 100K -> 100k (lowercase SI k)
- 100nf -> 100nF
- 69 symbols across all 6 boards (ASN-41, ARC-51A, APN-153, PDU,
  Gateway_Bridge, PanelGroup_Base). ERC 0/0 on all.

No functional/footprint/LCSC change. PDU generic 10k and precision
divider 10k now both read "10k", distinguished by tolerance (1% vs 0.1%).
Parts:
- R22, R23, R24, R25, R26, R27, R28, R29, R30, R31, R32, R33, R42, R43, R44, R5: value 10K -> 10k
Changed lines of the file:
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@@
 			)
 		)
-		(property "Value" "10K"
+		(property "Value" "10k"
 			(at 193.04 50.8 90)
 			(show_name no)
@@
 			)
 		)
-		(property "Value" "10K"
+		(property "Value" "10k"
 			(at 238.76 95.25 90)
 			(hide yes)
@@
 			)
 		)
-		(property "Value" "10K"
+		(property "Value" "10k"
 			(at 231.14 95.25 90)
 			(hide yes)
@@
 			)
 		)
-		(property "Value" "10K"
+		(property "Value" "10k"
 			(at 241.3 39.37 90)
 			(show_name no)
@@
 			)
 		)
-		(property "Value" "10K"
+		(property "Value" "10k"
 			(at 83.82 135.89 90)
 			(show_name no)
@@
 			)
 		)
-		(property "Value" "10K"
+		(property "Value" "10k"
 			(at 146.05 95.25 90)
 			(show_name no)
@@
 			)
 		)
-		(property "Value" "10K"
+		(property "Value" "10k"
 			(at 193.04 40.64 90)
 			(show_name no)
@@
 			)
 		)
-		(property "Value" "10K"
+		(property "Value" "10k"
 			(at 43.2436 69.2893 90)
 			(show_name no)
@@
 			)
 		)
-		(property "Value" "10K"
+		(property "Value" "10k"
 			(at 83.82 146.05 90)
 			(show_name no)
@@
 			)
 		)
-		(property "Value" "10K"
+		(property "Value" "10k"
 			(at 146.05 50.8 90)
 			(show_name no)
@@
 			)
 		)
-		(property "Value" "10K"
+		(property "Value" "10k"
 			(at 236.22 100.33 0)
 			(show_name no)
@@
 			)
 		)
-		(property "Value" "10K"
+		(property "Value" "10k"
 			(at 146.05 40.64 90)
 			(show_name no)
@@
 			)
 		)
-		(property "Value" "10K"
+		(property "Value" "10k"
 			(at 146.05 85.09 90)
 			(show_name no)
@@
 			)
 		)
-		(property "Value" "10K"
+		(property "Value" "10k"
 			(at 83.82 140.97 90)
 			(show_name no)
@@
 			)
 		)
-		(property "Value" "10K"
+		(property "Value" "10k"
 			(at 127 134.62 90)
 			(show_name no)
@@
 			)
 		)
-		(property "Value" "10K"
+		(property "Value" "10k"
 			(at 241.3 49.53 90)
 			(show_name no)

Commit message: refactor(pcb): consolidate ceramic 10uF to single 35V part
The 10uF ceramic 0805 caps were split across two SKUs — C669099 (25V)
and C49010152 (35V) — distinguished only by rail. Standardize all 8
ceramic positions to the 35V part (C49010152); 35V covers the 25V
positions and collapses the BOM to one ceramic 10uF value.

Electrolytic 10uF (C3343) unchanged. Aluminum-bulk replacement deferred
to a future round. 8 caps across all 6 boards, ERC 0/0.
Parts:
- C2: LCSC C669099 -> C49010152; Rating 25V -> 35V
Changed lines of the file:
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@@
 			)
 		)
-		(property "LCSC" "C669099"
+		(property "LCSC" "C49010152"
 			(at 0 0 0)
 			(hide yes)
@@
 			)
 		)
-		(property "Rating" "25V"
+		(property "Rating" "35V"
 			(at 0 0 0)
 			(hide yes)

Commit message: fix(pcb): right-size MCP23017/TCA9548 bulk 10uF->1uF (ARC/APN)
The 10uF ceramic bulk beside the MCP23017 and TCA9548 (ARC C2/C20,
APN C2) is oversized: both are low-current I2C parts whose datasheets
call for only 0.1uF, already present. Drop to 1uF (reuse C28323, 0805
unchanged) — keeps ample bulk, frees the 10uF/35V ceramic. No footprint
or symbol change; ERC clean.
Parts:
- C2: value 10uF -> 1uF; LCSC C49010152 -> C28323; Rating 35V -> 50V; Tolerance 20% -> 10%
Changed lines of the file:
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@@
 			)
 		)
-		(property "Value" "10uF"
+		(property "Value" "1uF"
 			(at 58.42 35.5662 0)
 			(show_name no)
@@
 			)
 		)
-		(property "LCSC" "C49010152"
+		(property "LCSC" "C28323"
 			(at 0 0 0)
 			(hide yes)
@@
 			)
 		)
-		(property "Tolerance" "20%"
+		(property "Tolerance" "10%"
 			(at 0 0 0)
 			(hide yes)
@@
 			)
 		)
-		(property "Rating" "35V"
+		(property "Rating" "50V"
 			(at 0 0 0)
 			(hide yes)

Commit message: feat(pcb): add descriptive IPN field to all on-board symbols (#238 Phase 3) (#239)
Phase 3 of the IPN convention (#238): adds a stable, descriptive
**Internal Part Number** to every on-board symbol, co-equal with LCSC.
BOMs now anchor on a fixed identity; the LCSC can change with
availability without altering the part's identity.

## What changed
- **352 symbols** across all 6 boards (multi-sheet aware) get an `IPN`
field. **51 distinct IPNs.** ERC clean fleet-wide.
- **Off-board controls** (encoders/switches/pots/OLED/stepper — no
footprint, connector-coupled) get **no IPN**, per the standing off-board
exclusion. On-board modules (RP2040-ZERO) and the RESET tact switch
**do** get IPNs.
- `.gitignore`: FreeCAD backups (`*.FCBak`/`*.FCStd1`) + KiCad ERC/DRC
reports (`*-erc.rpt`/`*-drc.rpt`).

## Scheme (descriptive, locked in #238)
`RES-10K-1PCT-0805` · `CAP-CER-100NF-50V-0805` · `CAP-ELEC-22UF-16V-D4`
· `IC-STM32F103C8-LQFP` · `CONN-XH-8P` · `TVS-SMBJ12A-SMB` ·
`FUSE-HOLDER-BLADE-DIP4` · `SW-TACT-6MM` · `MOD-RP2040-ZERO`.

Resolved the 3 open encoding items: ferrite → `FB-600R-0805` (TDK
600Ω@100MHz), NTC → `NTC-10K-1206` (APV 10K), fuse holder (C19727305 is
a *holder*, not a fuse) → one `FUSE-HOLDER-BLADE-DIP4`.

## Not in this PR (later phases of #238)
- **Phase 2 — InvenTree:** set the IPN field + link SupplierParts incl
backorder alternates (one IPN → many LCSC). This is what actually
delivers the churn-proofing; needs reviewed InvenTree writes.
- **Phase 4 — order flow:** resolve IPN → in-stock LCSC at order time.

Refs #238.
Parts:
- C1: IPN (none) -> CAP-CER-100NF-50V-0805
- C2: IPN (none) -> CAP-CER-1UF-50V-0805
- R22, R23, R24, R25, R26, R27, R28, R29, R30, R31, R32, R33, R42, R43, R44, R5: IPN (none) -> RES-10K-1PCT-0805
- R3: IPN (none) -> RES-100R-1PCT-0805
- U1: IPN (none) -> IC-MCP23017-SSOP
Changed lines of the file:
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@@
 			)
 		)
+		(property "IPN" "RES-10K-1PCT-0805"
+			(at 193.04 48.26 0)
+			(hide yes)
+			(show_name no)
+			(do_not_autoplace no)
+			(effects
+				(font
+					(size 1.27 1.27)
+				)
+			)
+		)
 		(property "Description" "Resistor, small symbol"
 			(at 193.04 48.26 0)
@@
 			)
 		)
+		(property "IPN" "RES-10K-1PCT-0805"
+			(at 236.22 95.25 0)
+			(hide yes)
+			(show_name no)
+			(do_not_autoplace no)
+			(effects
+				(font
+					(size 1.27 1.27)
+				)
+			)
+		)
 		(property "Description" "Resistor, small symbol"
 			(at 236.22 95.25 0)
@@
 			)
 		)
+		(property "IPN" "CAP-CER-1UF-50V-0805"
+			(at 55.88 34.29 0)
+			(hide yes)
+			(show_name no)
+			(do_not_autoplace no)
+			(effects
+				(font
+					(size 1.27 1.27)
+				)
+			)
+		)
 		(property "Description" "Unpolarized capacitor, small symbol"
 			(at 55.88 34.29 0)
@@
 			)
 		)
+		(property "IPN" "RES-10K-1PCT-0805"
+			(at 233.68 95.25 0)
+			(hide yes)
+			(show_name no)
+			(do_not_autoplace no)
+			(effects
+				(font
+					(size 1.27 1.27)
+				)
+			)
+		)
 		(property "Description" "Resistor, small symbol"
 			(at 233.68 95.25 0)
@@
 			)
 		)
+		(property "IPN" "RES-10K-1PCT-0805"
+			(at 241.3 41.91 0)
+			(hide yes)
+			(show_name no)
+			(do_not_autoplace no)
+			(effects
+				(font
+					(size 1.27 1.27)
+				)
+			)
+		)
 		(property "Description" "Resistor, small symbol"
 			(at 241.3 41.91 0)
@@
 			)
 		)
+		(property "IPN" "RES-10K-1PCT-0805"
+			(at 81.28 135.89 0)
+			(hide yes)
+			(show_name no)
+			(do_not_autoplace no)
+			(effects
+				(font
+					(size 1.27 1.27)
+				)
+			)
+		)
 		(property "Description" "Resistor, small symbol"
 			(at 81.28 135.89 0)
@@
 			)
 		)
+		(property "IPN" "RES-10K-1PCT-0805"
+			(at 146.05 92.71 0)
+			(hide yes)
+			(show_name no)
+			(do_not_autoplace no)
+			(effects
+				(font
+					(size 1.27 1.27)
+				)
+			)
+		)
 		(property "Description" "Resistor, small symbol"
 			(at 146.05 92.71 0)
@@
 			)
 		)
+		(property "IPN" "CAP-CER-100NF-50V-0805"
+			(at 43.18 34.29 0)
+			(hide yes)
+			(show_name no)
+			(do_not_autoplace no)
+			(effects
+				(font
+					(size 1.27 1.27)
+				)
+			)
+		)
 		(property "Description" "Unpolarized capacitor, small symbol"
 			(at 43.18 34.29 0)
@@
 			)
 		)
+		(property "IPN" "RES-100R-1PCT-0805"
+			(at 43.18 59.69 0)
+			(hide yes)
+			(show_name no)
+			(do_not_autoplace no)
+			(effects
+				(font
+					(size 1.27 1.27)
+				)
+			)
+		)
 		(property "Description" "Resistor, small symbol"
 			(at 43.18 59.69 0)
@@
 			)
 		)
+		(property "IPN" "RES-10K-1PCT-0805"
+			(at 193.04 43.18 0)
+			(hide yes)
+			(show_name no)
+			(do_not_autoplace no)
+			(effects
+				(font
+					(size 1.27 1.27)
+				)
+			)
+		)
 		(property "Description" "Resistor, small symbol"
 			(at 193.04 43.18 0)
@@
 			)
 		)
+		(property "IPN" "RES-10K-1PCT-0805"
+			(at 43.18 67.31 0)
+			(hide yes)
+			(show_name no)
+			(do_not_autoplace no)
+			(effects
+				(font
+					(size 1.27 1.27)
+				)
+			)
+		)
 		(property "Description" "Resistor, small symbol"
 			(at 43.18 67.31 0)
@@
 			)
 		)
+		(property "IPN" "RES-10K-1PCT-0805"
+			(at 81.28 146.05 0)
+			(hide yes)
+			(show_name no)
+			(do_not_autoplace no)
+			(effects
+				(font
+					(size 1.27 1.27)
+				)
+			)
+		)
 		(property "Description" "Resistor, small symbol"
 			(at 81.28 146.05 0)
@@
 			)
 		)
+		(property "IPN" "RES-10K-1PCT-0805"
+			(at 146.05 48.26 0)
+			(hide yes)
+			(show_name no)
+			(do_not_autoplace no)
+			(effects
+				(font
+					(size 1.27 1.27)
+				)
+			)
+		)
 		(property "Description" "Resistor, small symbol"
 			(at 146.05 48.26 0)
@@
 			)
 		)
+		(property "IPN" "IC-MCP23017-SSOP"
+			(at 68.58 92.71 0)
+			(hide yes)
+			(show_name no)
+			(do_not_autoplace no)
+			(effects
+				(font
+					(size 1.27 1.27)
+				)
+				(justify left)
+			)
+		)
 		(property "Description" "16-bit I/O expander, I2C, interrupts, w pull-ups, SSOP-28"
 			(at 63.5 64.77 0)
@@
 			)
 		)
+		(property "IPN" "RES-10K-1PCT-0805"
+			(at 238.76 95.25 0)
+			(hide yes)
+			(show_name no)
+			(do_not_autoplace no)
+			(effects
+				(font
+					(size 1.27 1.27)
+				)
+			)
+		)
 		(property "Description" "Resistor, small symbol"
 			(at 238.76 95.25 0)
@@
 			)
 		)
+		(property "IPN" "RES-10K-1PCT-0805"
+			(at 146.05 43.18 0)
+			(hide yes)
+			(show_name no)
+			(do_not_autoplace no)
+			(effects
+				(font
+					(size 1.27 1.27)
+				)
+			)
+		)
 		(property "Description" "Resistor, small symbol"
 			(at 146.05 43.18 0)
@@
 			)
 		)
+		(property "IPN" "RES-10K-1PCT-0805"
+			(at 146.05 87.63 0)
+			(hide yes)
+			(show_name no)
+			(do_not_autoplace no)
+			(effects
+				(font
+					(size 1.27 1.27)
+				)
+			)
+		)
 		(property "Description" "Resistor, small symbol"
 			(at 146.05 87.63 0)
@@
 			)
 		)
+		(property "IPN" "RES-10K-1PCT-0805"
+			(at 81.28 140.97 0)
+			(hide yes)
+			(show_name no)
+			(do_not_autoplace no)
+			(effects
+				(font
+					(size 1.27 1.27)
+				)
+			)
+		)
 		(property "Description" "Resistor, small symbol"
 			(at 81.28 140.97 0)
@@
 			)
 		)
+		(property "IPN" "RES-10K-1PCT-0805"
+			(at 127 137.16 0)
+			(hide yes)
+			(show_name no)
+			(do_not_autoplace no)
+			(effects
+				(font
+					(size 1.27 1.27)
+				)
+			)
+		)
 		(property "Description" "Resistor, small symbol"
 			(at 127 137.16 0)
@@
 			(at 241.3 46.99 0)
 			(hide yes)
+			(show_name no)
+			(do_not_autoplace no)
+			(effects
+				(font
+					(size 1.27 1.27)
+				)
+			)
+		)
+		(property "IPN" "RES-10K-1PCT-0805"
+			(at 241.3 46.99 0)
+			(hide yes)
