File: PCB/Right_Console/Right_Navigation/ARC-51A_UHF/ARC-51A_UHF.kicad_sch (KiCad schematic)
At the start: 0 parts

Commit message: feat(pcb): ARC-51A_UHF B2 schematic — Right_Nav UHF radio breakout
AN/ARC-51A UHF radio control panel breakout (#185), Right_Navigation NODE 2.
I2C-class sub-panel, no MCU — routes to the ASN-41 host over I2C2.

- MCP23017 @0x20: 4 DIR encoders (freq/preset) + XMIT 3-pos one-hot + SQUELCH;
  INTA push-pull -> J pin6, INTB NC.
- TCA9548A @0x71 -> 3 OLEDs (2x 1.3" freq + 1x 0.91" channel), all 0x3C.
- MODE 4-pos analog ladder + VOL pot -> host ADC (pins 7/8); RC host-side.
- J_ARC51A_I2C 8-pin (both-end 33/100 ohm termination) + J_BL 2-pin
  (backlight strings deferred to B4).
- Part props: 1% CRCW0805 resistors + stocked 50V/25V caps (InvenTree reuse).

ERC clean (0 violations). Firmware mux-arbitration carry-item logged in #172.
Parts:
- added H1, H2, H3, H4, H5, H6, H7, H8: MountingHole, MountingHole:MountingHole_2.7mm_M2.5, symbol Mechanical:MountingHole
- added J9: J_ARC51A_I2C, Connector_JST:JST_XH_B8B-XH-A_1x08_P2.50mm_Vertical, symbol Connector_Generic:Conn_01x08
- added R54, R55: 33, Resistor_SMD:R_0805_2012Metric, symbol Device:R
Connections:
- new net: J9.1 (Pin_1), R55.2
- new net: J9.2 (Pin_2), R54.1
- new net +3.3V: J9.5 (Pin_5)
- new net ARC51_MODE: J9.7 (Pin_7)
- new net GND: J9.3 (Pin_3), J9.4 (Pin_4)
- new net I2C2_SCL: R54.2
- new net I2C2_SDA: R55.1
- new net INT_A2: J9.6 (Pin_6)
- new net VOL: J9.8 (Pin_8)
Other:
- added sheet Backlight (Backlight.kicad_sch)
- added sheet OLEDs (OLEDs.kicad_sch)
- added sheet Switches (Switches.kicad_sch)

Commit message: feat(pcb): label LCSC/tolerance/voltage across fleet boards (Right_Nav + PDU + base) (#235)
Populates **LCSC part number + tolerance + voltage** fields across all
six fleet boards, so each schematic drives an orderable BOM.

## Boards labeled (ERC 0/0 on all)
- **Right_Nav:** ASN-41, ARC-51A, APN-153
- **Power:** PDU
- **Base:** Gateway_Bridge, PanelGroup_Base

## What it does
- LCSC + tolerance + voltage on every assembled part, corrected to the
selected part (100nF 50V, resistors 1%, AMS1117 C6186→C347222, 10µF
split 25V/35V by +12V rail).
- Off-board panel controls (encoders, rotary switches, OLED, pot,
stepper, MEM button) left blank — connector-coupled, no assembly LCSC.
- Pin headers hand-soldered; RP2040-Zero left blank (module, sourced
separately).

## Design corrections captured here
- **PDU 1k series/anti-alias → 1%** (C110774 0.1% → C844939): precision
belongs only on the divider ratio resistors (33k/13k/10k); the series 1k
sit into high-Z ADC pins where 1% is identical. Drops the precision part
from the board.
- **DESIGN-NOTES:** records the 1k downgrade + the order-time shunt
upgrade (C346481 ±100ppm → C500740 ±25ppm, drop-in 2512).

## Not in this PR (follow-ups)
- Fleet component **standardization** (10µF-bulk→electrolytic,
consolidate to single 35V value, IPN convention) — separate pass.
- InvenTree backfill of the new SKUs.
Parts:
- J9: LCSC (none) -> C23067548
- R54, R55: LCSC (none) -> C2090807
Changed lines of the file:
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@@
 			)
 		)
-		(property "LCSC" ""
+		(property "LCSC" "C2090807"
 			(at 229.87 307.34 0)
 			(hide yes)
@@
 			)
 		)
-		(property "LCSC" ""
+		(property "LCSC" "C23067548"
 			(at 229.87 307.34 0)
 			(hide yes)
@@
 			)
 		)
-		(property "LCSC" ""
-			(at 229.87 307.34 0)
-			(hide yes)
+		(property "LCSC" "C2090807"
+			(at 229.87 307.34 0)
+			(hide yes)

Commit message: feat(pcb): add descriptive IPN field to all on-board symbols (#238 Phase 3) (#239)
Phase 3 of the IPN convention (#238): adds a stable, descriptive
**Internal Part Number** to every on-board symbol, co-equal with LCSC.
BOMs now anchor on a fixed identity; the LCSC can change with
availability without altering the part's identity.

## What changed
- **352 symbols** across all 6 boards (multi-sheet aware) get an `IPN`
field. **51 distinct IPNs.** ERC clean fleet-wide.
- **Off-board controls** (encoders/switches/pots/OLED/stepper — no
footprint, connector-coupled) get **no IPN**, per the standing off-board
exclusion. On-board modules (RP2040-ZERO) and the RESET tact switch
**do** get IPNs.
- `.gitignore`: FreeCAD backups (`*.FCBak`/`*.FCStd1`) + KiCad ERC/DRC
reports (`*-erc.rpt`/`*-drc.rpt`).

## Scheme (descriptive, locked in #238)
`RES-10K-1PCT-0805` · `CAP-CER-100NF-50V-0805` · `CAP-ELEC-22UF-16V-D4`
· `IC-STM32F103C8-LQFP` · `CONN-XH-8P` · `TVS-SMBJ12A-SMB` ·
`FUSE-HOLDER-BLADE-DIP4` · `SW-TACT-6MM` · `MOD-RP2040-ZERO`.

Resolved the 3 open encoding items: ferrite → `FB-600R-0805` (TDK
600Ω@100MHz), NTC → `NTC-10K-1206` (APV 10K), fuse holder (C19727305 is
a *holder*, not a fuse) → one `FUSE-HOLDER-BLADE-DIP4`.

## Not in this PR (later phases of #238)
- **Phase 2 — InvenTree:** set the IPN field + link SupplierParts incl
backorder alternates (one IPN → many LCSC). This is what actually
delivers the churn-proofing; needs reviewed InvenTree writes.
- **Phase 4 — order flow:** resolve IPN → in-stock LCSC at order time.

Refs #238.
Parts:
- J9: IPN (none) -> CONN-XH-8P
- R54, R55: IPN (none) -> RES-33R-1PCT-0805
Changed lines of the file:
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@@
+			)
+		)
+		(property "IPN" "RES-33R-1PCT-0805"
+			(at 158.75 58.42 0)
+			(hide yes)
+			(show_name no)
+			(do_not_autoplace no)
+			(effects
+				(font
+					(size 1.27 1.27)
+				)
 			)
 		)
@@
 			)
 		)
+		(property "IPN" "CONN-XH-8P"
+			(at 143.51 36.83 0)
+			(hide yes)
+			(show_name no)
+			(do_not_autoplace no)
+			(effects
+				(font
+					(size 1.27 1.27)
+				)
+			)
+		)
 		(property "Description" "Generic connector, single row, 01x08, script generated (kicad-library-utils/schlib/autogen/connector/)"
 			(at 143.51 36.83 0)
@@
 			(at 156.21 58.42 0)
 			(hide yes)
+			(show_name no)
+			(do_not_autoplace no)
+			(effects
+				(font
+					(size 1.27 1.27)
+				)
+			)
+		)
+		(property "IPN" "RES-33R-1PCT-0805"
+			(at 156.21 58.42 0)
+			(hide yes)
